File: pcb_1/pcb_1.kicad_pcb (KiCad board)
At the start: 2 copper layers, 105.9 x 66.5 mm, 47 parts, among them J1 ACin, J2 Vout, J3 2N3055_conn, J4 DCin, P1 CONN_01X07, P2 CONN_01X01, P3 CONN_01X01, P4 CONN_01X01, P5 CONN_01X01, P6 CONN_01X01, P7 CONN_01X01, Q2 BD139, U1 MAX9944ASA+T, U2 MCP3422A0-E/SN, U3 MCP4822-E/SN, U4 TL072, U5 LM7705MM/NOPB, U6 SPX2920U-5.0, U7 LM317AT, U9 INA240A1PWR

Commit message: Footprintit lisätty ja pcb-layout aloitettu
Parts:
- removed Cb5, Cb7: 0.1u, Capacitors_SMD:C_0805_HandSoldering
- removed P1: CONN_01X07, Pin_Headers:Pin_Header_Straight_1x07_Pitch2.54mm
- removed P2, P3, P4, P5, P6, P7: CONN_01X01, Pin_Headers:Pin_Header_Straight_1x01_Pitch2.54mm
- added C10: 0.1u, Capacitors_SMD:C_0805_HandSoldering, F.Cu at (168.4, 31.1)
- added C11: 0.1u, Capacitors_SMD:C_0805_HandSoldering, F.Cu at (168.5, 20.8)
- added C12: 0.1u, Capacitors_SMD:C_0805_HandSoldering, F.Cu at (257.1, 42.0)
- added C13: 0.1u, Capacitors_SMD:C_0805_HandSoldering, F.Cu at (205.6, 24.1)
- added C14: 0.1u, Capacitors_SMD:C_0805_HandSoldering, F.Cu at (217.3, 47.7)
- added C15: C, Capacitors_SMD:C_0805_HandSoldering, F.Cu at (220.2, 58.7)
- added C16: 0.1u, Capacitors_SMD:C_0805_HandSoldering, F.Cu at (233.9, 48.4)
- added C17: 0.1u, Capacitors_SMD:C_0805_HandSoldering, F.Cu at (254.5, 30.8)
- added C8: C, Capacitors_SMD:C_0805_HandSoldering, F.Cu at (184.8, 43.4)
- added C9: 0.1u, Capacitors_SMD:C_0805_HandSoldering, F.Cu at (184.8, 45.4)
- added Cb2: 0.1u, Capacitors_SMD:C_0805_HandSoldering, F.Cu at (190.6, 41.8)
- added D4: D_Schottky, Diodes_SMD:D_PowerDI-123, F.Cu at (98.7, 121.4)
- added D5: Zener 15V, Diodes_THT:D_5W_P12.70mm_Horizontal, F.Cu at (62.6, 105.3)
- added D6: Zener 30V, Diodes_THT:D_5W_P12.70mm_Horizontal, F.Cu at (36.7, 100.8)
- added J5: Isolated_ISP, Pin_Headers:Pin_Header_Straight_1x08_Pitch2.54mm, F.Cu at (232.0, 19.9)
- added J6: AVR-ISP-6, Pin_Headers:Pin_Header_Straight_2x03_Pitch2.54mm, F.Cu at (261.0, 66.2)
- added J7: THERM0, Pin_Headers:Pin_Header_Straight_1x02_Pitch2.54mm, F.Cu at (275.8, 37.0)
- added J8: THERM1, Pin_Headers:Pin_Header_Straight_1x02_Pitch2.54mm, F.Cu at (275.5, 31.2)
- added J9: Screw_Terminal_01x01, Connectors:Banana_Jack_1Pin, F.Cu at (214.6, 131.4)
- added K1: DIPxx-1Axx-11x, lab_power_supply:PCJ-105D3MH, F.Cu at (27.8, 134.5)
- added Q1: BD139, TO_SOT_Packages_THT:TO-126_Vertical, F.Cu at (105.8, 127.0)
- added Q3: Q_NMOS_DGS, TO_SOT_Packages_SMD:SuperSOT-3, F.Cu at (245.5, 64.1)
- added Q4: Q_NMOS_DGS, TO_SOT_Packages_SMD:SuperSOT-3, F.Cu at (239.1, 60.2)
- added Q5: Q_NMOS_DGS, TO_SOT_Packages_SMD:SuperSOT-3, F.Cu at (239.8, 71.4)
- added Q6: Q_NMOS_DGS, TO_SOT_Packages_SMD:SuperSOT-3, F.Cu at (245.1, 68.6)
- added R10: 330, Resistors_SMD:R_0805_HandSoldering, F.Cu at (227.9, 23.8)
- added R11: 330, Resistors_SMD:R_0805_HandSoldering, F.Cu at (234.7, 38.0)
- added R12: 330, Resistors_SMD:R_0805_HandSoldering, F.Cu at (244.0, 51.2)
- added R13: 330, Resistors_SMD:R_0805_HandSoldering, F.Cu at (234.7, 24.7)
- added R14: 100, Resistors_SMD:R_0805_HandSoldering, F.Cu at (254.3, 65.8)
- added R15: 100, Resistors_SMD:R_0805_HandSoldering, F.Cu at (227.9, 58.3)
- added R16: 100, Resistors_SMD:R_0805_HandSoldering, F.Cu at (223.9, 38.2)
- added R17: 100, Resistors_SMD:R_0805_HandSoldering, F.Cu at (230.0, 40.1)
- added R18: 500, Resistors_SMD:R_0805_HandSoldering, F.Cu at (233.7, 32.3)
- added R19: R, Resistors_SMD:R_0805_HandSoldering, F.Cu at (271.3, 35.9)
- added R20: R, Resistors_SMD:R_0805_HandSoldering, F.Cu at (270.5, 32.3)
- added R21: 5k, Resistors_SMD:R_0805_HandSoldering, F.Cu at (217.2, 45.3)
- added R22: 5k, Resistors_SMD:R_0805_HandSoldering, F.Cu at (216.9, 51.1)
- added R23: 10k, Resistors_SMD:R_0805_HandSoldering, F.Cu at (223.8, 40.2)
- added TP1: UNREG, Measurement_Points:Measurement_Point_Round-SMD-Pad_Big, F.Cu at (220.3, 122.2)
- added TP2: DACa, Measurement_Points:Measurement_Point_Round-SMD-Pad_Big, F.Cu at (198.9, 38.4)
- added TP3: DACb, Measurement_Points:Measurement_Point_Round-SMD-Pad_Big, F.Cu at (197.9, 30.2)
- added U8: HCPL2601SD, lab_power_supply:HCPL2631SD, F.Cu at (246.1, 31.1)
- C1, C4, C6: value CONN_01X02 -> C; footprint Pin_Headers:Pin_Header_Straight_1x02_Pitch2.54mm -> Capacitors_SMD:C_0805_HandSoldering
- C2: value CONN_01X02 -> 10u; footprint Pin_Headers:Pin_Header_Straight_1x02_Pitch2.54mm -> Capacitors_THT:CP_Radial_D8.0mm_P5.00mm
- C3: value CONN_01X02 -> 0.1u; footprint Pin_Headers:Pin_Header_Straight_1x02_Pitch2.54mm -> Capacitors_SMD:C_0805_HandSoldering
- C5: value CONN_01X02 -> 0.22u; footprint Pin_Headers:Pin_Header_Straight_1x02_Pitch2.54mm -> Capacitors_SMD:C_0805_HandSoldering
- C7: value CONN_01X02 -> 100u; footprint Pin_Headers:Pin_Header_Straight_1x02_Pitch2.54mm -> Capacitors_THT:CP_Radial_D8.0mm_P5.00mm
- CP1: value 4700uF 50V -> 15000uF 50V
- Cb1, Cb3, Cb4, R5: moved to F.Cu
- D1: value D_Schottky -> D_Bridge_+AA-; footprint Diodes_SMD:D_0805 -> lab_power_supply:GBU6D_diode-bridge; moved to F.Cu
- D2: value Zener 15V -> Zener 5V; footprint Diodes_THT:D_5W_P12.70mm_Horizontal -> Diodes_THT:D_DO-41_SOD81_P7.62mm_Horizontal
- D3: value D_Bridge_+AA- -> Zener 25V; footprint lab_power_supply:GBU6D_diode-bridge -> Diodes_THT:D_5W_P12.70mm_Horizontal
- J1: value ACin -> Screw_Terminal_01x02; footprint Wire_Connections_Bridges:WireConnection_2.50mmDrill_LargePad -> Connectors:Banana_Jack_2Pin
- J2: value Vout -> Screw_Terminal_01x02; footprint Wire_Connections_Bridges:WireConnection_2.50mmDrill_LargePad -> Connectors:Banana_Jack_2Pin
- J3: value 2N3055_conn -> Conn_01x02_Male; footprint Wire_Connections_Bridges:WireConnection_2.50mmDrill_LargePad -> Pin_Headers:Pin_Header_Straight_1x02_Pitch2.54mm
- J4: value DCin -> Screw_Terminal_01x02; footprint Wire_Connections_Bridges:WireConnection_2.50mmDrill_LargePad -> Connectors:Banana_Jack_2Pin
- Q2: value BD139 -> Q_NMOS_DGS; footprint TO_SOT_Packages_THT:TO-126_Vertical -> TO_SOT_Packages_SMD:SuperSOT-3
- R1: value 2.2k -> 1k; moved to F.Cu
- R2: value 2.2k -> 10k; moved to F.Cu
- R3: value 15k -> R; moved to F.Cu
- R4: value 1.2k -> 2.2k; moved to F.Cu
- R6: value R -> 16k; moved to F.Cu
- R7: value R -> 1.3k; moved to F.Cu
- R8, R9: value R -> 1k; moved to F.Cu
- U1: value MAX9944ASA+T -> MAX9944; moved to F.Cu
- U2: value MCP3422A0-E/SN -> SPX2920U-5.0; footprint Housings_SOIC:SOIC-8_3.9x4.9mm_Pitch1.27mm -> Power_Integrations:TO-220; moved to F.Cu
- U3: value MCP4822-E/SN -> INA240A1PWR; moved to F.Cu
- U4: value TL072 -> MCP4822-E/SN; footprint Housings_DIP:DIP-8_W7.62mm_Socket_LongPads -> Housings_SOIC:SOIC-8_3.9x4.9mm_Pitch1.27mm
- U5: value LM7705MM/NOPB -> MCP3422A0-E/SN; footprint Housings_SSOP:MSOP-8_3x3mm_Pitch0.65mm -> Housings_SOIC:SOIC-8_3.9x4.9mm_Pitch1.27mm; moved to F.Cu
- U6: value SPX2920U-5.0 -> HCPL2631SD; footprint Power_Integrations:TO-220 -> lab_power_supply:HCPL2631SD
- U7: value LM317AT -> HCPL2631SD; footprint Power_Integrations:TO-220 -> lab_power_supply:HCPL2631SD
- U9: value INA240A1PWR -> ATmega328PB-AU; footprint Housings_SOIC:SOIC-8_3.9x4.9mm_Pitch1.27mm -> Housings_QFP:TQFP-32_7x7mm_Pitch0.8mm; moved to F.Cu
- moved J1 230.3 mm to (267.8, 122.6), turned to 90 degrees
- moved F1 159.5 mm to (235.7, 91.9), turned to 0 degrees
- moved CP1 151.8 mm to (208.5, 103.6), turned to 90 degrees
- moved J3 144.3 mm to (27.3, 139.1), turned to 270 degrees
- moved D1 142.2 mm to (244.9, 112.1), turned to 0 degrees
- moved U7 136.0 mm to (254.6, 50.7)
- moved U6 115.3 mm to (215.0, 23.9), turned to 0 degrees
- moved Q2 114.0 mm to (240.0, 66.9), turned to 0 degrees
- moved Rs1 113.4 mm to (62.6, 138.4), turned to 180 degrees
- moved D2 105.0 mm to (205.5, 70.9), turned to 90 degrees
- moved R2 97.5 mm to (209.8, 66.8), turned to 90 degrees
- moved U9 97.4 mm to (225.7, 48.0), turned to 0 degrees
- moved R1 97.3 mm to (210.3, 74.1), turned to 90 degrees
- moved Cb3 91.2 mm to (180.7, 37.1), turned to 0 degrees
- moved Cb4 90.8 mm to (180.7, 39.8), turned to 0 degrees
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Connections:
- C1 pad 1: +5V -> Vmon
- C1 pad 2: GND -> Net-(C1-Pad2)
- C2 pad 2: GND -> GNDA
- C3 pad 1: Net-(C3-Pad1) -> Net-(C2-Pad1)
- C3 pad 2: Net-(C3-Pad2) -> GNDA
- C4 pad 1: -0.232V -> Net-(C4-Pad1)
- C4 pad 2: GND -> Imon
- C5 pad 2: GND -> GNDA
- C6 pad 1: Net-(C6-Pad1) -> +5V
- C6 pad 2: Net-(C6-Pad2) -> GNDA
- C7 pad 1: Net-(C7-Pad1) -> +5V
- C7 pad 2: Net-(C7-Pad2) -> GNDA
- CP1 pad 2: GND -> GNDA
- Cb1 pad 1: GND -> +5V
- Cb1 pad 2: +5V -> GNDA
- Cb3 pad 1: Net-(Cb3-Pad1) -> GNDA
- Cb3 pad 2: GND -> Net-(Cb3-Pad2)
- Cb4 pad 1: Net-(Cb4-Pad1) -> GNDA
- Cb4 pad 2: GND -> Net-(Cb4-Pad2)
- D1 pad 1: Net-(C7-Pad1) -> Net-(CP1-Pad1)
- D2 pad 1: Net-(CP1-Pad1) -> UNREG_MON
- D2 pad 2: Net-(D2-Pad2) -> GNDA
- D3 pad 1: Net-(CP1-Pad1) -> Net-(C2-Pad1)
- D3 pad 2: Net-(D3-Pad2) -> GNDA
- F1 pad 1: Net-(D3-Pad2) -> Net-(D1-Pad2)
- J1 pad 1: Net-(F1-Pad2) -> Net-(D1-Pad3)
- J1 pad 2: Net-(D3-Pad3) -> Net-(F1-Pad2)
- J2 pad 1: GND -> Net-(J2-Pad1)
- J4 pad 1: Net-(CP1-Pad1) -> Net-(D6-Pad1)
- J4 pad 2: GND -> GNDA
- Q2 pad 1: Net-(J3-Pad2) -> Net-(Q2-Pad1)
- Q2 pad 2: Net-(CP1-Pad1) -> Net-(J5-Pad4)
- Q2 pad 3: Net-(Q2-Pad3) -> Net-(C12-Pad2)
- R1 pad 1: Net-(D1-Pad2) -> Net-(CP1-Pad1)
- R1 pad 2: Net-(C6-Pad2) -> UNREG_MON
- R2 pad 1: Net-(Q2-Pad3) -> UNREG_MON
- R2 pad 2: Net-(D1-Pad2) -> GNDA
- R3 pad 1: Net-(J2-Pad2) -> Net-(CP1-Pad1)
- R3 pad 2: Net-(C6-Pad1) -> Net-(C2-Pad1)
- R4 pad 1: Net-(C6-Pad1) -> Net-(D4-Pad2)
- R4 pad 2: GND -> Net-(C1-Pad2)
- R5 pad 1: Net-(R5-Pad1) -> Net-(Q1-Pad3)
- R5 pad 2: current_limiter -> Net-(D4-Pad2)
- R6 pad 1: GND -> Net-(K1-Pad1)
- R6 pad 2: Net-(Cb5-Pad1) -> Vmon
- R7 pad 1: Net-(Cb5-Pad1) -> Vmon
- R7 pad 2: -0.232V -> GNDA
- R8 pad 1: Net-(R8-Pad1) -> Iset
- R8 pad 2: GND -> Net-(Cb3-Pad2)
- R9 pad 1: Net-(C2-Pad1) -> Vset
- R9 pad 2: Net-(R8-Pad1) -> Net-(Cb4-Pad2)
- Rs1 pad 1: Net-(J3-Pad1) -> Net-(J2-Pad2)
- Rs1 pad 2: Net-(J2-Pad2) -> Net-(K1-Pad1)
- U1 pad 1: Net-(C6-Pad2) -> Net-(C1-Pad2)
- U1 pad 2: Net-(C6-Pad1) -> Vmon
- U1 pad 3: Net-(Cb3-Pad1) -> Vset
- U1 pad 4: GND -> GNDA
- U1 pad 5: Net-(Cb4-Pad1) -> Iset
- U1 pad 6: Net-(C7-Pad2) -> Imon
- U1 pad 7: Net-(C7-Pad1) -> Net-(C4-Pad1)
- U2 pad 1: Net-(C6-Pad1) -> Net-(C5-Pad1)
- U2 pad 2: GND -> GNDA
- U3 pad 1: +5V -> Net-(K1-Pad1)
- U3 pad 2: DAC_cs -> GNDA
- U3 pad 3: DAC_sck -> GNDA
- U3 pad 4: DAC_sdi -> Net-(U3-Pad4)
- U3 pad 5: Net-(Cb5-Pad1) -> Imon
- U3 pad 6: Net-(Cb4-Pad1) -> +5V
- U3 pad 7: Net-(Cb5-Pad1) -> GNDA
- U3 pad 8: Net-(Cb3-Pad1) -> Net-(J2-Pad2)
- U4 pad 1: Net-(R5-Pad1) -> +5V
- U4 pad 2: Net-(C7-Pad1) -> DAC_CS
- U4 pad 3: Net-(D1-Pad2) -> DAC_SCK
- U4 pad 4: GND -> DAC_SDI
- U4 pad 5: (no net) -> DAC_LDAC
- U4 pad 6: (no net) -> Net-(Cb3-Pad2)
- U4 pad 7: (no net) -> GNDA
- U4 pad 8: +5V -> Net-(Cb4-Pad2)
- U5 pad 1: Net-(C3-Pad1) -> Vmon
- U5 pad 2: GND -> GNDA
- U5 pad 3: GND -> +5V
- U5 pad 4: +5V -> ADC_SDA
- U5 pad 5: GND -> ADC_SCL
- U5 pad 6: -0.232V -> GNDA
- U5 pad 7: Net-(C5-Pad1) -> Imon
- U5 pad 8: Net-(C3-Pad2) -> GNDA
- U6 pad 1: Net-(D2-Pad2) -> Net-(Q3-Pad1)
- U6 pad 2: GND -> Net-(C12-Pad2)
- U6 pad 3: +5V -> Net-(C12-Pad2)
- U7 pad 1: Net-(R8-Pad1) -> Net-(Q5-Pad1)
- U7 pad 2: Net-(C2-Pad1) -> Net-(C12-Pad2)
- U7 pad 3: Net-(CP1-Pad1) -> Net-(C12-Pad2)
- U9 pad 1: Net-(J2-Pad2) -> Net-(U9-Pad1)
- U9 pad 2: GND -> Net-(U9-Pad2)
- U9 pad 3: GND -> ADC_SDA
- U9 pad 4: Net-(U9-Pad4) -> +5V
- U9 pad 5: Net-(C7-Pad2) -> GNDD
- U9 pad 6: +5V -> ADC_SCL
- U9 pad 7: GND -> Net-(U9-Pad7)
- U9 pad 8: Net-(J3-Pad1) -> Net-(U9-Pad8)
Routing:
- net GND: track 739.2 -> 0.00 mm, vias 9 -> 0
- net Net-(CP1-Pad1): track 176.1 -> 0.00 mm
- net +5V: track 149.4 -> 0.00 mm, vias 4 -> 0
- net current_limiter: track 103.1 -> 0.00 mm
- net Net-(Cb3-Pad1): track 91.4 -> 0.00 mm, vias 2 -> 0
- net Net-(C6-Pad1): track 88.7 -> 0.00 mm, vias 2 -> 0
- net Net-(C7-Pad2): track 75.8 -> 0.00 mm, vias 2 -> 0
- net Net-(Cb4-Pad1): track 69.6 -> 0.00 mm, vias 2 -> 0
- net Net-(J2-Pad2): track 44.3 -> 0.00 mm
- net Net-(C2-Pad1): track 28.6 -> 0.00 mm
- net Net-(D3-Pad3): track 27.3 -> 0.00 mm
- net Net-(J3-Pad1): track 27.0 -> 0.00 mm
- net Net-(Cb5-Pad1): track 26.0 -> 0.00 mm
- net Net-(C7-Pad1): track 25.8 -> 0.00 mm
- net Net-(C6-Pad2): track 21.6 -> 0.00 mm
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- removed copper zone on B.Cu, net GND
- removed copper zone on F.Cu, net GND
Other:
- board outline removed

Commit message: Komponentit aseteltu paikoilleen ja vähän traceja vedelty
Parts:
- removed J9: Screw_Terminal_01x01, Connectors:Banana_Jack_1Pin
- J1, J4: footprint Connectors:Banana_Jack_2Pin -> Connectors_Terminal_Blocks:TerminalBlock_bornier-2_P5.08mm
- J2: value Screw_Terminal_01x02 -> Screw_Terminal_01x03; footprint Connectors:Banana_Jack_2Pin -> Connectors_Terminal_Blocks:TerminalBlock_bornier-3_P5.08mm
- Rs1: footprint Resistors_THT:R_Axial_DIN0414_L11.9mm_D4.5mm_P25.40mm_Horizontal -> Resistors_SMD:R_2816; moved to B.Cu
- moved TP2 146.3 mm to (52.8, 45.4)
- moved C17 133.3 mm to (121.4, 37.7), turned to 0 degrees
- moved TP3 129.4 mm to (69.3, 45.5)
- moved Cb3 123.6 mm to (57.2, 41.4)
- moved C12 121.0 mm to (137.4, 60.5), turned to 180 degrees
- moved U8 120.1 mm to (126.9, 45.3)
- moved Q6 119.8 mm to (125.9, 57.3), turned to 180 degrees
- moved R8 115.7 mm to (58.4, 46.5), turned to 90 degrees
- moved Cb4 114.0 mm to (66.7, 41.8), turned to 180 degrees
- moved CP1 113.3 mm to (95.6, 94.5)
- moved C10 111.8 mm to (58.3, 51.0), turned to 180 degrees
- moved C8 111.7 mm to (74.0, 57.5), turned to 90 degrees
- moved R18 111.6 mm to (125.8, 60.6)
- moved Cb2 109.9 mm to (80.9, 47.5)
- moved C9 109.5 mm to (76.0, 57.5), turned to 270 degrees
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Connections:
- J2 pad 1: Net-(J2-Pad1) -> Net-(CP1-Pad1)
- Q1 pad 1: Net-(J2-Pad1) -> Net-(J2-Pad2)
- Rs1 pad 1: Net-(J2-Pad2) -> Net-(J2-Pad3)
- U3 pad 8: Net-(J2-Pad2) -> Net-(J2-Pad3)
Routing:
- net Net-(CP1-Pad1): track 0.00 -> 94.0 mm
- net Net-(K1-Pad1): track 0.00 -> 55.0 mm, vias 0 -> 1
- net Net-(D1-Pad3): track 0.00 -> 41.7 mm
- net Net-(J2-Pad3): track 0.00 -> 37.0 mm, vias 0 -> 1
- net Net-(J6-Pad5): track 0.00 -> 28.7 mm
- net Net-(D6-Pad1): track 0.00 -> 28.2 mm
- net Net-(J6-Pad4): track 0.00 -> 24.3 mm
- net Net-(F1-Pad2): track 0.00 -> 23.0 mm
- net Net-(J6-Pad3): track 0.00 -> 21.4 mm
- net Net-(J3-Pad2): track 0.00 -> 21.0 mm
- net Net-(J3-Pad1): track 0.00 -> 20.1 mm
- net Net-(J6-Pad1): track 0.00 -> 15.4 mm
- net Net-(D1-Pad2): track 0.00 -> 14.3 mm
- net GNDA: track 0.00 -> 13.8 mm
- net Net-(J2-Pad2): track 0.00 -> 11.5 mm
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