File: pcb_1/pcb_1.sch (KiCad schematic (older format))
At the start: 45 parts, among them J1 ACin, J2 Vout, J3 2N3055_conn, J4 DCin, P1 CONN_01X07, P2 CONN_01X01, P3 CONN_01X01, P4 CONN_01X01, P5 CONN_01X01, P6 CONN_01X01, P7 CONN_01X01, Q2 BD139, U1 MAX9944ASA+T, U2 MCP3422A0-E/SN, U3 MCP4822-E/SN, U4 TL072, U5 LM7705MM/NOPB, U6 SPX2920U-5.0, U7 LM317AT, U9 INA240A1PWR

Commit message: 30.10 syövytetty pcb
Parts:
- added R6, R7: 27k, Resistors_SMD:R_0805_HandSoldering, symbol R
- R3: value 15k -> 16k
- R4: value 1.2k -> 1.3k
Connections:
- net -0.232V: now also R7.2; no longer Cb5.1, P4.1 (P1), U3.5 (LDAC), U3.7 (VSS)
- net GND: now also R6.1
- net at C7.2 (P2), P6.1 (P1), U2.7 (CH2+)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: now also U1.6 (INB-); no longer U1.5 (INB+)
- net at Cb4.1, P3.1 (P1), U3.6 (VoutB): now also U1.5 (INB+); no longer U1.6 (INB-)
- new net: Cb5.1, P4.1 (P1), R6.2, R7.1, U3.5 (LDAC), U3.7 (VSS)
Other:
- moved on the sheet: P4, P6
Changed lines of the file:
@@
 P 9400 4700
 F 0 "R3" V 9480 4700 50  0000 C CNN
-F 1 "15k" V 9400 4700 50  0000 C CNN
+F 1 "16k" V 9400 4700 50  0000 C CNN
 F 2 "Resistors_SMD:R_0805_HandSoldering" V 9330 4700 50  0001 C CNN
 F 3 "" H 9400 4700 50  0000 C CNN
@@
 P 9400 5200
 F 0 "R4" V 9480 5200 50  0000 C CNN
-F 1 "1.2k" V 9400 5200 50  0000 C CNN
+F 1 "1.3k" V 9400 5200 50  0000 C CNN
 F 2 "Resistors_SMD:R_0805_HandSoldering" V 9330 5200 50  0001 C CNN
 F 3 "" H 9400 5200 50  0000 C CNN
@@
 Text GLabel 8400 4700 2    60   Output ~ 0
 -0.232V
-Text GLabel 4950 2050 2    60   Input ~ 0
+Text GLabel 5300 2300 2    60   Input ~ 0
 -0.232V
 $Comp
@@
 L CONN_01X01 P6
 U 1 1 5DAB3A4E
-P 8250 3050
-F 0 "P6" H 8250 3150 50  0000 C CNN
-F 1 "CONN_01X01" V 8350 3050 50  0000 C CNN
-F 2 "Pin_Headers:Pin_Header_Straight_1x01_Pitch2.54mm" H 8250 3050 50  0001 C CNN
-F 3 "" H 8250 3050 50  0000 C CNN
-	1    8250 3050
-	1    0    0    -1
+P 8550 2900
+F 0 "P6" H 8550 3000 50  0000 C CNN
+F 1 "CONN_01X01" V 8650 2900 50  0000 C CNN
+F 2 "Pin_Headers:Pin_Header_Straight_1x01_Pitch2.54mm" H 8550 2900 50  0001 C CNN
+F 3 "" H 8550 2900 50  0000 C CNN
+	1    8550 2900
+	0    1    1    0
 $EndComp
 $Comp
@@
 L CONN_01X01 P4
 U 1 1 5DAB40D2
-P 8900 4950
-F 0 "P4" H 8900 5050 50  0000 C CNN
-F 1 "CONN_01X01" V 9000 4950 50  0000 C CNN
-F 2 "Pin_Headers:Pin_Header_Straight_1x01_Pitch2.54mm" H 8900 4950 50  0001 C CNN
-F 3 "" H 8900 4950 50  0000 C CNN
-	1    8900 4950
+P 5250 2050
+F 0 "P4" H 5250 2150 50  0000 C CNN
+F 1 "CONN_01X01" V 5350 2050 50  0000 C CNN
+F 2 "Pin_Headers:Pin_Header_Straight_1x01_Pitch2.54mm" H 5250 2050 50  0001 C CNN
+F 3 "" H 5250 2050 50  0000 C CNN
+	1    5250 2050
 	1    0    0    -1
 $EndComp
@@
 Connection ~ 7700 1800
 Wire Wire Line
-	7800 3100 7800 2700
-Wire Wire Line
-	7800 2700 7550 2700
+	7550 2700 10000 2700
 Wire Wire Line
 	10450 1800 10450 3000
-Wire Wire Line
-	7550 2800 10000 2800
 Wire Wire Line
 	5350 900  5350 1250
@@
 Wire Wire Line
 	4300 3250 4300 4500
-Connection ~ 8000 2800
 Wire Wire Line
 	7750 4700 8400 4700
@@
 	4800 2150 4800 2050
 Wire Wire Line
-	4650 2050 4950 2050
+	4650 2050 5050 2050
 Connection ~ 4800 2050
-Wire Wire Line
-	8300 4950 8700 4950
-Connection ~ 8300 4950
 Connection ~ 10450 2700
 Wire Wire Line
@@
 Wire Wire Line
 	7700 2600 7550 2600
-Wire Wire Line
-	8000 2600 8000 3250
 Wire Wire Line
 	6350 2950 6350 2700
@@
 	8300 3400 8300 3350
 Connection ~ 8300 3350
-Wire Wire Line
-	8050 3050 8000 3050
-Connection ~ 8000 3050
 Wire Wire Line
 	7500 2050 7550 2050
@@
 	9100 3650 8950 3650
 Wire Wire Line
-	10000 2800 10000 3750
+	10000 2700 10000 3750
 Wire Wire Line
 	8950 3650 8950 3550
@@
 	1    0    0    -1
 $EndComp
+Wire Wire Line
+	7800 3100 7800 2800
+Wire Wire Line
+	7800 2800 7550 2800
+Connection ~ 8550 2700
+Wire Wire Line
+	8000 2600 8000 3250
+Connection ~ 8000 2700
+$Comp
+L R R7
+U 1 1 5DB99C16
+P 5050 2200
+F 0 "R7" V 5130 2200 50  0000 C CNN
+F 1 "27k" V 5050 2200 50  0000 C CNN
+F 2 "Resistors_SMD:R_0805_HandSoldering" V 4980 2200 50  0001 C CNN
+F 3 "" H 5050 2200 50  0000 C CNN
+	1    5050 2200
+	1    0    0    -1
+$EndComp
+$Comp
+L R R6
+U 1 1 5DB99C95
+P 5050 1900
+F 0 "R6" V 5130 1900 50  0000 C CNN
+F 1 "27k" V 5050 1900 50  0000 C CNN
+F 2 "Resistors_SMD:R_0805_HandSoldering" V 4980 1900 50  0001 C CNN
+F 3 "" H 5050 1900 50  0000 C CNN
+	1    5050 1900
+	1    0    0    -1
+$EndComp
+Wire Wire Line
+	5300 2300 5150 2300
+Wire Wire Line
+	5150 2300 5150 2350
+Wire Wire Line
+	5150 2350 5050 2350
+$Comp
+L GND #PWR031
+U 1 1 5DB9A0A5
+P 5150 1600
+F 0 "#PWR031" H 5150 1350 50  0001 C CNN
+F 1 "GND" H 5150 1450 50  0000 C CNN
+F 2 "" H 5150 1600 50  0000 C CNN
+F 3 "" H 5150 1600 50  0000 C CNN
+	1    5150 1600
+	1    0    0    -1
+$EndComp
+Wire Wire Line
+	5150 1600 5150 1500
+Wire Wire Line
+	5150 1500 5050 1500
+Wire Wire Line
+	5050 1500 5050 1750
 $EndSCHEMATC

Commit message: pcb: Add first version with a MCU
Also update the Kicad project to Kicad version 5
Parts:
- removed C1, C2, C3, C4, C5, C6, C7: CONN_01X02, Pin_Headers:Pin_Header_Straight_1x02_Pitch2.54mm, symbol CONN_01X02
- removed Cb7: 0.1u, Capacitors_SMD:C_0805_HandSoldering, symbol C
- removed J1: ACin, Wire_Connections_Bridges:WireConnection_2.50mmDrill_LargePad, symbol Screw_Terminal_1x02
- removed J2: Vout, Wire_Connections_Bridges:WireConnection_2.50mmDrill_LargePad, symbol Screw_Terminal_1x02
- removed J3: 2N3055_conn, Wire_Connections_Bridges:WireConnection_2.50mmDrill_LargePad, symbol Screw_Terminal_1x02
- removed J4: DCin, Wire_Connections_Bridges:WireConnection_2.50mmDrill_LargePad, symbol Screw_Terminal_1x02
- removed P1: CONN_01X07, Pin_Headers:Pin_Header_Straight_1x07_Pitch2.54mm, symbol CONN_01X07
- removed P2, P3, P4, P5, P6, P7: CONN_01X01, Pin_Headers:Pin_Header_Straight_1x01_Pitch2.54mm, symbol CONN_01X01
- removed Q2: BD139, TO_SOT_Packages_THT:TO-126_Vertical, symbol BD139
- removed R5: 2.2k, Resistors_SMD:R_0805_HandSoldering, symbol R
- removed R6, R7: 27k, Resistors_SMD:R_0805_HandSoldering, symbol R
- removed R8, R9: R, Resistors_SMD:R_0805_HandSoldering, symbol R
- removed U1: MAX9944ASA+T, Housings_SOIC:SOIC-8_3.9x4.9mm_Pitch1.27mm, symbol MAX9944ASA+T
- removed U4: TL072, Housings_DIP:DIP-8_W7.62mm_Socket_LongPads, symbol OP275
- removed U5: LM7705MM/NOPB, Housings_SSOP:MSOP-8_3x3mm_Pitch0.65mm, symbol LM7705MM/NOPB
- removed U7: LM317AT, Power_Integrations:TO-220, symbol LM317AT
- added C1: CP, symbol Device:CP
- added C2, C3, C4: C, symbol Device:C
- added C?: 0.1u, symbol Device:C
- added C?: 10u, symbol Device:CP
- added J1, J2, J3: Screw_Terminal_01x02, symbol Connector:Screw_Terminal_01x02
- added Q1: BD139, Package_TO_SOT_THT:TO-126-3_Vertical, symbol Transistor_BJT:BD139
- added U1: MAX9944, symbol lab_power_supply:MAX9944
- CP1: symbol CP -> Device:CP
- Cb1, Cb3, Cb4, Cb5: symbol C -> Device:C
- D1: symbol D_Schottky -> Device:D_Schottky
- D2: symbol D_Zener -> Device:D_Zener
- D3: symbol D_Bridge_+AA- -> Device:D_Bridge_+AA-
- F1: symbol Fuse -> Device:Fuse
- R1, R2, R3, R4, Rs1: symbol R -> Device:R
- U2: symbol MCP3422A0-E/SN -> lab_power_supply:MCP3422A0-E_SN
- U3: symbol MCP4822-E/SN -> lab_power_supply:MCP4822-E_SN
- U6: symbol SPX2920U-5.0 -> lab_power_supply:SPX2920U-5.0
- U9: symbol INA240A1PWR -> lab_power_supply:INA240A1PWR
Connections:
- net labels added: +28V, DAC_ldac, GNDA, Imon, Iset, Vmon, Vset
- net labels removed: -0.232V, Charge_pump, GND, OP_AMP, current_limiter
- wire segments 132 -> 108
Other:
- moved on the sheet: CP1, Cb1, Cb3, Cb4, Cb5, D1, D2, D3, F1, R1, R2, R3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

Commit message: pcb: Add relay and filtering capacitors
Parts:
- added C? (x2): C, symbol Device:C
- added C?: 10u, symbol Device:CP
- added D?: Zener 30V, symbol Device:D_Zener
- added D?: Zener 5V, symbol Device:D_Zener
- added J?: Conn_01x02_Male, symbol Connector:Conn_01x02_Male
- added K?: AZ850-x, Relay_THT:Relay_DPDT_FRT5, symbol Relay:AZ850-x
- added R?: 1k, symbol Device:R
- added R?: 10k, symbol Device:R
- added R? (x2): R, symbol Device:R
- added TP?: TestPoint, symbol Connector:TestPoint
- C1: value CP -> 10u
- C2: value C -> 0.1u
- CP1: value 4700uF 50V -> 15000uF 50V
Connections:
- net labels added: UNREG_MON
- net labels removed: +28V
- wire segments 108 -> 140
- no-connect marks 0 -> 2
Other:
- moved on the sheet: C1, C2, C3, C4, C?, CP1, Cb1, Cb3, Cb4, Cb5, D1, D2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

Commit message: pcb: Fix mismatching global labels
Also add connections for thermistors.
Parts:
- removed K?: AZ850-x, Relay_THT:Relay_DPDT_FRT5, symbol Relay:AZ850-x
- added K1: DIPxx-1Axx-11x, Relay_THT:Relay_StandexMeder_DIP_LowProfile, symbol Relay:DIPxx-1Axx-11x
- added TP2: DACa, symbol Connector:TestPoint
- added TP3: DACb, symbol Connector:TestPoint
- C8, C9: renamed from C?; value C -> 0.1u
- R7, R8: renamed from R?; value R -> 1k
- TP1: renamed from TP?; value TestPoint -> UNREG
- gave numbers to parts that had none: 8
- renumbered Cb5 to Cb2, D3 to D1, D1 to D3, D2 to D4, J3 to J1, J1 to J2, J2 to J4, R1 to R3, R2 to R4, R3 to R5, R4 to R6, U6 to U2, U9 to U3, U3 to U4, U2 to U5
Connections:
- net labels added: ADC_SCL, ADC_SDA, DAC_CS, DAC_LDAC, DAC_SCK, DAC_SDI
- net labels removed: ADC_scl, ADC_sda, DAC_cs, DAC_ldac, DAC_sck, DAC_sdi
- wire segments 140 -> 145
- no-connect marks 2 -> 0
Other:
- moved on the sheet: C8, C9, D5, R7, R8

Commit message: pcb: Add Zener regulator to op-amp supply
Parts:
- added C5: 0.22u, symbol Device:C
- added C7: 100u, symbol Device:CP
- added D3: Zener 25V, symbol Device:D_Zener
- added R3: R, symbol Device:R
- renumbered C3 to C1, C8 to C10, C9 to C11, C1 to C2, C2 to C3, C5 to C6, C6 to C8, C7 to C9, D3 to D4, D4 to D5, D5 to D6, R3 to R4, R4 to R5, R5 to R6, R6 to R7, R7 to R8, R8 to R9
Connections:
- wire segments 145 -> 156
Other:
- moved on the sheet: C2, C3, C6, Cb1, D5, U2

Commit message: Footprintit lisätty ja pcb-layout aloitettu
Parts:
- removed C6, C8: 10u, symbol Device:CP
- added C6, C8: C, Capacitors_SMD:C_0805_HandSoldering, symbol Device:C
- added J9: Screw_Terminal_01x01, Connectors:Banana_Jack_1Pin, symbol Connector:Screw_Terminal_01x01
- C1, C10, C11, C3, C4, C5, C9: footprint (none) -> Capacitors_SMD:C_0805_HandSoldering
- C2, C7: footprint (none) -> Capacitors_THT:CP_Radial_D8.0mm_P5.00mm
- D2: footprint (none) -> Diodes_THT:D_DO-41_SOD81_P7.62mm_Horizontal
- D3, D6: footprint (none) -> Diodes_THT:D_5W_P12.70mm_Horizontal
- D4: footprint Diodes_SMD:D_0805 -> Diodes_SMD:D_PowerDI-123
- J1, J2, J4: footprint (none) -> Connectors:Banana_Jack_2Pin
- J3: footprint (none) -> Pin_Headers:Pin_Header_Straight_1x02_Pitch2.54mm
- K1: footprint Relay_THT:Relay_StandexMeder_DIP_LowProfile -> lab_power_supply:PCJ-105D3MH
- Q1: footprint Package_TO_SOT_THT:TO-126-3_Vertical -> TO_SOT_Packages_THT:TO-126_Vertical
- R1, R2, R3, R8, R9: footprint (none) -> Resistors_SMD:R_0805_HandSoldering
- TP1, TP2, TP3: footprint (none) -> Measurement_Points:Measurement_Point_Round-SMD-Pad_Big
- U1: footprint (none) -> Housings_SOIC:SOIC-8_3.9x4.9mm_Pitch1.27mm
Connections:
- wire segments 156 -> 158
Changed lines of the file:
@@
 EESchema Schematic File Version 4
-LIBS:pcb_1-cache
 EELAYER 30 0
 EELAYER END
@@
 F 0 "D4" H 7450 2150 50  0000 C CNN
 F 1 "D_Schottky" H 7350 1950 50  0000 C CNN
-F 2 "Diodes_SMD:D_0805" H 7450 2050 50  0001 C CNN
+F 2 "Diodes_SMD:D_PowerDI-123" H 7450 2050 50  0001 C CNN
 F 3 "" H 7450 2050 50  0000 C CNN
 	1    7450 2050
@@
 F 0 "Q1" H 8292 1796 50  0000 L CNN
 F 1 "BD139" H 8292 1705 50  0000 L CNN
-F 2 "Package_TO_SOT_THT:TO-126-3_Vertical" H 8300 1675 50  0001 L CIN
+F 2 "TO_SOT_Packages_THT:TO-126_Vertical" H 8300 1675 50  0001 L CIN
 F 3 "http://www.st.com/internet/com/TECHNICAL_RESOURCES/TECHNICAL_LITERATURE/DATASHEET/CD00001225.pdf" H 8100 1750 50  0001 L CNN
 	1    8100 1750
@@
 F 0 "J2" H 8480 2292 50  0000 L CNN
 F 1 "Screw_Terminal_01x02" H 8480 2201 50  0000 L CNN
-F 2 "" H 8400 2300 50  0001 C CNN
+F 2 "Connectors:Banana_Jack_2Pin" H 8400 2300 50  0001 C CNN
 F 3 "~" H 8400 2300 50  0001 C CNN
 	1    8400 2300
@@
 F 0 "J4" H 11030 5242 50  0000 L CNN
 F 1 "Screw_Terminal_01x02" H 11030 5151 50  0000 L CNN
-F 2 "" H 10950 5250 50  0001 C CNN
+F 2 "Connectors:Banana_Jack_2Pin" H 10950 5250 50  0001 C CNN
 F 3 "~" H 10950 5250 50  0001 C CNN
 	1    10950 5250
@@
 F 0 "U1" H 6750 2050 50  0000 C CNN
 F 1 "MAX9944" H 6750 1950 50  0000 C CNN
-F 2 "" H 6650 1750 50  0001 C CNN
+F 2 "Housings_SOIC:SOIC-8_3.9x4.9mm_Pitch1.27mm" H 6650 1750 50  0001 C CNN
 F 3 "http://www.ti.com/lit/ds/symlink/lm358.pdf" H 6650 1750 50  0001 C CNN
 	1    6650 1750
@@
 F 0 "U1" H 5308 2096 50  0000 L CNN
 F 1 "MAX9944" H 5308 2005 50  0000 L CNN
-F 2 "" H 5350 2050 50  0001 C CNN
+F 2 "Housings_SOIC:SOIC-8_3.9x4.9mm_Pitch1.27mm" H 5350 2050 50  0001 C CNN
 F 3 "http://www.ti.com/lit/ds/symlink/lm358.pdf" H 5350 2050 50  0001 C CNN
 	3    5350 2050
@@
 F 0 "C1" V 6600 2100 50  0000 C CNN
 F 1 "C" V 6600 1900 50  0000 C CNN
-F 2 "" H 6688 1850 50  0001 C CNN
+F 2 "Capacitors_SMD:C_0805_HandSoldering" H 6688 1850 50  0001 C CNN
 F 3 "~" H 6650 2000 50  0001 C CNN
 	1    6650 2000
@@
 F 0 "J1" H 918 925 50  0000 C CNN
 F 1 "Screw_Terminal_01x02" H 918 1016 50  0000 C CNN
-F 2 "" H 1000 1250 50  0001 C CNN
+F 2 "Connectors:Banana_Jack_2Pin" H 1000 1250 50  0001 C CNN
 F 3 "~" H 1000 1250 50  0001 C CNN
 	1    1000 1250
@@
 F 0 "C3" H 5050 2150 50  0000 L CNN
 F 1 "0.1u" H 5050 1950 50  0000 L CNN
-F 2 "" H 5038 1900 50  0001 C CNN
+F 2 "Capacitors_SMD:C_0805_HandSoldering" H 5038 1900 50  0001 C CNN
 F 3 "~" H 5000 2050 50  0001 C CNN
 	1    5000 2050
@@
 F 0 "C2" H 4750 2150 50  0000 L CNN
 F 1 "10u" H 4750 1950 50  0000 L CNN
-F 2 "" H 4738 1900 50  0001 C CNN
+F 2 "Capacitors_THT:CP_Radial_D8.0mm_P5.00mm" H 4738 1900 50  0001 C CNN
 F 3 "~" H 4700 2050 50  0001 C CNN
 	1    4700 2050
@@
 	5000 2200 5000 2350
 Wire Wire Line
-	5250 1200 8200 1200
+	5250 1200 6100 1200
 Connection ~ 5250 1750
 Wire Wire Line
@@
 F 0 "C9" V 5300 5400 50  0000 C CNN
 F 1 "0.1u" V 5200 5350 50  0000 C CNN
-F 2 "" H 5488 5250 50  0001 C CNN
+F 2 "Capacitors_SMD:C_0805_HandSoldering" H 5488 5250 50  0001 C CNN
 F 3 "~" H 5450 5400 50  0001 C CNN
 	1    5450 5400
 	0    -1   -1   0
-$EndComp
-$Comp
-L Device:CP C8
-U 1 1 5DF4A4CB
-P 5450 5150
-F 0 "C8" V 5200 5100 50  0000 L CNN
-F 1 "10u" V 5300 5100 50  0000 L CNN
-F 2 "" H 5488 5000 50  0001 C CNN
-F 3 "~" H 5450 5150 50  0001 C CNN
-	1    5450 5150
-	0    1    1    0
 $EndComp
 Wire Wire Line
@@
 F 0 "D6" V 10404 5329 50  0000 L CNN
 F 1 "Zener 30V" V 10750 5100 50  0000 L CNN
-F 2 "" H 10450 5250 50  0001 C CNN
+F 2 "Diodes_THT:D_5W_P12.70mm_Horizontal" H 10450 5250 50  0001 C CNN
 F 3 "~" H 10450 5250 50  0001 C CNN
 	1    10450 5250
@@
 F 0 "J3" V 9662 3894 50  0000 L CNN
 F 1 "Conn_01x02_Male" V 9753 3894 50  0000 L CNN
-F 2 "" H 9600 3850 50  0001 C CNN
+F 2 "Pin_Headers:Pin_Header_Straight_1x02_Pitch2.54mm" H 9600 3850 50  0001 C CNN
 F 3 "~" H 9600 3850 50  0001 C CNN
 	1    9600 3850
@@
 F 0 "TP1" H 5308 1318 50  0000 L CNN
 F 1 "UNREG" H 5308 1227 50  0000 L CNN
-F 2 "" H 5450 1200 50  0001 C CNN
+F 2 "Measurement_Points:Measurement_Point_Round-SMD-Pad_Big" H 5450 1200 50  0001 C CNN
 F 3 "~" H 5450 1200 50  0001 C CNN
 	1    5250 1200
@@
 F 0 "R1" H 2320 1396 50  0000 L CNN
 F 1 "1k" H 2320 1305 50  0000 L CNN
-F 2 "" V 2180 1350 50  0001 C CNN
+F 2 "Resistors_SMD:R_0805_HandSoldering" V 2180 1350 50  0001 C CNN
 F 3 "~" H 2250 1350 50  0001 C CNN
 	1    2250 1350
@@
 F 0 "R2" H 2320 1796 50  0000 L CNN
 F 1 "10k" H 2320 1705 50  0000 L CNN
-F 2 "" V 2180 1750 50  0001 C CNN
+F 2 "Resistors_SMD:R_0805_HandSoldering" V 2180 1750 50  0001 C CNN
 F 3 "~" H 2250 1750 50  0001 C CNN
 	1    2250 1750
@@
 F 0 "D2" V 2554 1829 50  0000 L CNN
 F 1 "Zener 5V" V 2645 1829 50  0000 L CNN
-F 2 "" H 2600 1750 50  0001 C CNN
+F 2 "Diodes_THT:D_DO-41_SOD81_P7.62mm_Horizontal" H 2600 1750 50  0001 C CNN
 F 3 "~" H 2600 1750 50  0001 C CNN
 	1    2600 1750
@@
 	2600 1900 2250 1900
 Connection ~ 2250 1900
-Wire Wire Line
-	4550 3300 4900 3300
 Connection ~ 2650 6400
 Connection ~ 2450 6200
@@
 F 0 "C4" V 6700 2750 50  0000 C CNN
 F 1 "C" V 6700 2950 50  0000 C CNN
-F 2 "" H 6688 2700 50  0001 C CNN
+F 2 "Capacitors_SMD:C_0805_HandSoldering" H 6688 2700 50  0001 C CNN
 F 3 "~" H 6650 2850 50  0001 C CNN
 	1    6650 2850
@@
 F 0 "U1" H 6750 2900 50  0000 C CNN
 F 1 "MAX9944" H 6750 2800 50  0000 C CNN
-F 2 "" H 6650 2600 50  0001 C CNN
+F 2 "Housings_SOIC:SOIC-8_3.9x4.9mm_Pitch1.27mm" H 6650 2600 50  0001 C CNN
 F 3 "http://www.ti.com/lit/ds/symlink/lm358.pdf" H 6650 2600 50  0001 C CNN
 	2    6650 2600
@@
 Wire Wire Line
 	7450 2200 7450 2600
-$Comp
-L Device:CP C6
-U 1 1 5DF40B6F
-P 4900 3450
-F 0 "C6" H 5018 3496 50  0000 L CNN
-F 1 "10u" H 5018 3405 50  0000 L CNN
-F 2 "" H 4938 3300 50  0001 C CNN
-F 3 "~" H 4900 3450 50  0001 C CNN
-	1    4900 3450
-	1    0    0    -1
-$EndComp
 Wire Wire Line
 	2250 1200 3550 1200
@@
 F 0 "K1" V 8983 4900 50  0000 C CNN
 F 1 "DIPxx-1Axx-11x" V 9074 4900 50  0000 C CNN
-F 2 "Relay_THT:Relay_StandexMeder_DIP_LowProfile" H 9900 4850 50  0001 L CNN
+F 2 "lab_power_supply:PCJ-105D3MH" H 9900 4850 50  0001 L CNN
 F 3 "https://standexelectronics.com/wp-content/uploads/datasheet_reed_relay_DIP.pdf" H 9550 4900 50  0001 C CNN
 	1    9550 4900
@@
 F 0 "C11" H 3285 6504 50  0000 R CNN
 F 1 "0.1u" H 3285 6595 50  0000 R CNN
-F 2 "" H 3438 6400 50  0001 C CNN
+F 2 "Capacitors_SMD:C_0805_HandSoldering" H 3438 6400 50  0001 C CNN
 F 3 "~" H 3400 6550 50  0001 C CNN
 	1    3400 6550
@@
 F 0 "R9" V 3350 6400 50  0000 C CNN
 F 1 "1k" V 3250 6400 50  0000 C CNN
-F 2 "" V 3080 6400 50  0001 C CNN
+F 2 "Resistors_SMD:R_0805_HandSoldering" V 3080 6400 50  0001 C CNN
 F 3 "~" H 3150 6400 50  0001 C CNN
 	1    3150 6400
@@
 F 0 "C10" H 3515 6096 50  0000 L CNN
 F 1 "0.1u" H 3515 6005 50  0000 L CNN
-F 2 "" H 3438 5900 50  0001 C CNN
+F 2 "Capacitors_SMD:C_0805_HandSoldering" H 3438 5900 50  0001 C CNN
 F 3 "~" H 3400 6050 50  0001 C CNN
 	1    3400 6050
@@
 F 0 "R8" V 2943 6200 50  0000 C CNN
 F 1 "1k" V 3034 6200 50  0000 C CNN
-F 2 "" V 3080 6200 50  0001 C CNN
+F 2 "Resistors_SMD:R_0805_HandSoldering" V 3080 6200 50  0001 C CNN
 F 3 "~" H 3150 6200 50  0001 C CNN
 	1    3150 6200
@@
 F 0 "TP2" H 2650 6350 50  0000 L CNN
 F 1 "DACa" H 2650 6250 50  0000 L CNN
-F 2 "" H 3050 6200 50  0001 C CNN
+F 2 "Measurement_Points:Measurement_Point_Round-SMD-Pad_Big" H 3050 6200 50  0001 C CNN
 F 3 "~" H 3050 6200 50  0001 C CNN
 	1    2850 6200
@@
 F 0 "TP3" H 2650 6550 50  0000 L CNN
 F 1 "DACb" H 2650 6450 50  0000 L CNN
-F 2 "" H 3050 6400 50  0001 C CNN
+F 2 "Measurement_Points:Measurement_Point_Round-SMD-Pad_Big" H 3050 6400 50  0001 C CNN
 F 3 "~" H 3050 6400 50  0001 C CNN
 	1    2850 6400
@@
 F 0 "C5" H 3350 3500 50  0000 L CNN
 F 1 "0.22u" H 3200 3400 50  0000 L CNN
-F 2 "" H 3588 3300 50  0001 C CNN
+F 2 "Capacitors_SMD:C_0805_HandSoldering" H 3588 3300 50  0001 C CNN
 F 3 "~" H 3550 3450 50  0001 C CNN
 	1    3550 3450
@@
 Wire Wire Line
 	3550 3700 4050 3700
-Wire Wire Line
-	4900 3300 5300 3300
-Connection ~ 4900 3300
 Wire Wire Line
 	5300 3700 4900 3700
@@
 F 0 "C7" H 5418 3496 50  0000 L CNN
 F 1 "100u" H 5418 3405 50  0000 L CNN
-F 2 "" H 5338 3300 50  0001 C CNN
+F 2 "Capacitors_THT:CP_Radial_D8.0mm_P5.00mm" H 5338 3300 50  0001 C CNN
 F 3 "~" H 5300 3450 50  0001 C CNN
 	1    5300 3450
@@
 F 0 "R3" H 5320 1446 50  0000 L CNN
 F 1 "R" H 5320 1355 50  0000 L CNN
-F 2 "" V 5180 1400 50  0001 C CNN
+F 2 "Resistors_SMD:R_0805_HandSoldering" V 5180 1400 50  0001 C CNN
 F 3 "~" H 5250 1400 50  0001 C CNN
 	1    5250 1400
@@
 F 0 "D3" V 4400 1850 50  0000 L CNN
 F 1 "Zener 25V" V 4500 1600 50  0000 L CNN
-F 2 "" H 4450 2050 50  0001 C CNN
+F 2 "Diodes_THT:D_5W_P12.70mm_Horizontal" H 4450 2050 50  0001 C CNN
 F 3 "~" H 4450 2050 50  0001 C CNN
 	1    4450 2050
@@
 $EndComp
 Connection ~ 4450 1750
+$Comp
+L Device:C C8
+U 1 1 5DD0A10F
+P 5450 5150
+F 0 "C8" V 5198 5150 50  0000 C CNN
+F 1 "C" V 5289 5150 50  0000 C CNN
+F 2 "Capacitors_SMD:C_0805_HandSoldering" H 5488 5000 50  0001 C CNN
+F 3 "~" H 5450 5150 50  0001 C CNN
+	1    5450 5150
+	0    1    1    0
+$EndComp
+$Comp
+L Device:C C6
+U 1 1 5DD21243
+P 4900 3450
+F 0 "C6" H 5015 3496 50  0000 L CNN
+F 1 "C" H 5015 3405 50  0000 L CNN
+F 2 "Capacitors_SMD:C_0805_HandSoldering" H 4938 3300 50  0001 C CNN
+F 3 "~" H 4900 3450 50  0001 C CNN
+	1    4900 3450
+	1    0    0    -1
+$EndComp
+Wire Wire Line
+	4550 3300 4900 3300
+Connection ~ 4900 3300
+Wire Wire Line
+	4900 3300 5300 3300
+$Comp
+L Connector:Screw_Terminal_01x01 J9
+U 1 1 5DD4748F
+P 6300 850
+F 0 "J9" H 6380 892 50  0000 L CNN
+F 1 "Screw_Terminal_01x01" H 6380 801 50  0000 L CNN
+F 2 "Connectors:Banana_Jack_1Pin" H 6300 850 50  0001 C CNN
+F 3 "~" H 6300 850 50  0001 C CNN
+	1    6300 850
+	1    0    0    -1
+$EndComp
+Wire Wire Line
+	6100 850  6100 1200
+Connection ~ 6100 1200
+Wire Wire Line
+	6100 1200 8200 1200
 $EndSCHEMATC
