File: pcb_1/pcb_1.sch (KiCad schematic (older format))
At the start: 48 parts, among them J1 Screw_Terminal_01x02, J2 Screw_Terminal_01x02, J3 Conn_01x02_Male, J4 Screw_Terminal_01x02, J9 Screw_Terminal_01x01, K1 DIPxx-1Axx-11x, Q1 BD139, U1 MAX9944, U2 SPX2920U-5.0, U3 INA240A1PWR, U4 MCP4822-E/SN, U5 MCP3422A0-E/SN

Commit message: Komponentit aseteltu paikoilleen ja vähän traceja vedelty
Parts:
- removed J2: Screw_Terminal_01x02, Connectors:Banana_Jack_2Pin, symbol Connector:Screw_Terminal_01x02
- removed J9: Screw_Terminal_01x01, Connectors:Banana_Jack_1Pin, symbol Connector:Screw_Terminal_01x01
- added J2: Screw_Terminal_01x03, Connectors_Terminal_Blocks:TerminalBlock_bornier-3_P5.08mm, symbol Connector:Screw_Terminal_01x03
- J1, J4: footprint Connectors:Banana_Jack_2Pin -> Connectors_Terminal_Blocks:TerminalBlock_bornier-2_P5.08mm
- Rs1: footprint Resistors_THT:R_Axial_DIN0414_L11.9mm_D4.5mm_P25.40mm_Horizontal -> Resistors_SMD:R_2816
Connections:
- wire segments 158 -> 162
Changed lines of the file:
@@
 F 0 "Rs1" V 8280 3800 50  0000 C CNN
 F 1 "0.1" V 8200 3800 50  0000 C CNN
-F 2 "Resistors_THT:R_Axial_DIN0414_L11.9mm_D4.5mm_P25.40mm_Horizontal" V 8130 3800 50  0001 C CNN
+F 2 "Resistors_SMD:R_2816" V 8130 3800 50  0001 C CNN
 F 3 "" H 8200 3800 50  0000 C CNN
 	1    8200 3800
@@
 $EndComp
 $Comp
-L Connector:Screw_Terminal_01x02 J2
-U 1 1 5DCB6E99
-P 8400 2300
-F 0 "J2" H 8480 2292 50  0000 L CNN
-F 1 "Screw_Terminal_01x02" H 8480 2201 50  0000 L CNN
-F 2 "Connectors:Banana_Jack_2Pin" H 8400 2300 50  0001 C CNN
-F 3 "~" H 8400 2300 50  0001 C CNN
-	1    8400 2300
-	1    0    0    -1
-$EndComp
-$Comp
 L Connector:Screw_Terminal_01x02 J4
 U 1 1 5DCB7E83
@@
 F 0 "J4" H 11030 5242 50  0000 L CNN
 F 1 "Screw_Terminal_01x02" H 11030 5151 50  0000 L CNN
-F 2 "Connectors:Banana_Jack_2Pin" H 10950 5250 50  0001 C CNN
+F 2 "Connectors_Terminal_Blocks:TerminalBlock_bornier-2_P5.08mm" H 10950 5250 50  0001 C CNN
 F 3 "~" H 10950 5250 50  0001 C CNN
 	1    10950 5250
@@
 F 0 "J1" H 918 925 50  0000 C CNN
 F 1 "Screw_Terminal_01x02" H 918 1016 50  0000 C CNN
-F 2 "Connectors:Banana_Jack_2Pin" H 1000 1250 50  0001 C CNN
+F 2 "Connectors_Terminal_Blocks:TerminalBlock_bornier-2_P5.08mm" H 1000 1250 50  0001 C CNN
 F 3 "~" H 1000 1250 50  0001 C CNN
 	1    1000 1250
@@
 Wire Wire Line
 	4900 3300 5300 3300
-$Comp
-L Connector:Screw_Terminal_01x01 J9
-U 1 1 5DD4748F
-P 6300 850
-F 0 "J9" H 6380 892 50  0000 L CNN
-F 1 "Screw_Terminal_01x01" H 6380 801 50  0000 L CNN
-F 2 "Connectors:Banana_Jack_1Pin" H 6300 850 50  0001 C CNN
-F 3 "~" H 6300 850 50  0001 C CNN
-	1    6300 850
-	1    0    0    -1
-$EndComp
 Wire Wire Line
 	6100 850  6100 1200
@@
 Wire Wire Line
 	6100 1200 8200 1200
+$Comp
+L Connector:Screw_Terminal_01x03 J2
+U 1 1 5DE7FCEE
+P 8700 2300
+F 0 "J2" H 8780 2342 50  0000 L CNN
+F 1 "Screw_Terminal_01x03" H 8780 2251 50  0000 L CNN
+F 2 "Connectors_Terminal_Blocks:TerminalBlock_bornier-3_P5.08mm" H 8700 2300 50  0001 C CNN
+F 3 "~" H 8700 2300 50  0001 C CNN
+	1    8700 2300
+	1    0    0    -1
+$EndComp
+Wire Wire Line
+	6100 850  8500 850
+Wire Wire Line
+	8500 850  8500 2200
+Wire Wire Line
+	8200 2300 8500 2300
+Wire Wire Line
+	8500 2400 8200 2400
 $EndSCHEMATC

Commit message: pcb: Releen ohjauspiiri lisätty
Parts:
- removed J3: Conn_01x02_Male, Pin_Headers:Pin_Header_Straight_1x02_Pitch2.54mm, symbol Connector:Conn_01x02_Male
- added D7: D, Diodes_THT:D_DO-41_SOD81_P7.62mm_Horizontal, symbol Device:D
- added J3: Conn_Relay, Pin_Headers:Pin_Header_Straight_1x03_Pitch2.54mm, symbol lab_power_supply:Conn_Relay
- added Q7: Q_NMOS_DGS, TO_SOT_Packages_SMD:SuperSOT-3, symbol Device:Q_NMOS_DGS
- added R24: 100k, Resistors_SMD:R_0805_HandSoldering, symbol Device:R
Connections:
- wire segments 162 -> 170
Changed lines of the file:
@@
 EESchema Schematic File Version 4
+LIBS:pcb_1-cache
 EELAYER 30 0
 EELAYER END
@@
 	7850 5500 7850 5650
 $Comp
-L Connector:Conn_01x02_Male J3
-U 1 1 5DD767CF
-P 9600 3850
-F 0 "J3" V 9662 3894 50  0000 L CNN
-F 1 "Conn_01x02_Male" V 9753 3894 50  0000 L CNN
-F 2 "Pin_Headers:Pin_Header_Straight_1x02_Pitch2.54mm" H 9600 3850 50  0001 C CNN
-F 3 "~" H 9600 3850 50  0001 C CNN
-	1    9600 3850
-	0    1    1    0
-$EndComp
-Wire Wire Line
-	9600 4200 9600 4050
-Wire Wire Line
-	9500 4050 9500 4200
-Wire Wire Line
-	9250 4700 9200 4700
-Wire Wire Line
-	9200 4700 9200 4200
-Wire Wire Line
-	9200 4200 9500 4200
-Wire Wire Line
-	9850 4700 9900 4700
-Wire Wire Line
-	9900 4700 9900 4200
-Wire Wire Line
-	9900 4200 9600 4200
-$Comp
 L Connector:TestPoint TP1
 U 1 1 5DDB2288
@@
 Wire Wire Line
 	8500 2400 8200 2400
+$Comp
+L Device:Q_NMOS_DGS Q7
+U 1 1 5DD62A9A
+P 10250 3800
+F 0 "Q7" H 10456 3754 50  0000 L CNN
+F 1 "Q_NMOS_DGS" H 10456 3845 50  0000 L CNN
+F 2 "TO_SOT_Packages_SMD:SuperSOT-3" H 10450 3900 50  0001 C CNN
+F 3 "~" H 10250 3800 50  0001 C CNN
+	1    10250 3800
+	1    0    0    1
+$EndComp
+Wire Wire Line
+	10350 4700 9850 4700
+Wire Wire Line
+	8950 4700 9250 4700
+Wire Wire Line
+	10350 3450 10350 3600
+$Comp
+L Device:R R24
+U 1 1 5DDF700F
+P 9900 3600
+F 0 "R24" H 9970 3646 50  0000 L CNN
+F 1 "100k" H 9970 3555 50  0000 L CNN
+F 2 "Resistors_SMD:R_0805_HandSoldering" V 9830 3600 50  0001 C CNN
+F 3 "~" H 9900 3600 50  0001 C CNN
+	1    9900 3600
+	1    0    0    -1
+$EndComp
+Connection ~ 9900 3450
+Wire Wire Line
+	9900 3450 10350 3450
+Wire Wire Line
+	10050 3800 9900 3800
+Wire Wire Line
+	9900 3800 9900 3750
+Wire Wire Line
+	9900 3800 9300 3800
+Wire Wire Line
+	9300 3800 9300 3550
+Wire Wire Line
+	9300 3550 8950 3550
+Connection ~ 9900 3800
+Wire Wire Line
+	8950 3450 9900 3450
+$Comp
+L lab_power_supply:Conn_Relay J3
+U 1 1 5DE25C13
+P 8750 3550
+F 0 "J3" H 8743 3233 50  0000 C CNN
+F 1 "Conn_Relay" H 8743 3324 50  0000 C CNN
+F 2 "Pin_Headers:Pin_Header_Straight_1x03_Pitch2.54mm" H 8750 3550 50  0001 C CNN
+F 3 "~" H 8750 3550 50  0001 C CNN
+	1    8750 3550
+	-1   0    0    1
+$EndComp
+$Comp
+L Device:D D7
+U 1 1 5DE2784A
+P 9550 4200
+F 0 "D7" H 9550 4416 50  0000 C CNN
+F 1 "D" H 9550 4325 50  0000 C CNN
+F 2 "Diodes_THT:D_DO-41_SOD81_P7.62mm_Horizontal" H 9550 4200 50  0001 C CNN
+F 3 "~" H 9550 4200 50  0001 C CNN
+	1    9550 4200
+	1    0    0    -1
+$EndComp
+Wire Wire Line
+	8950 3650 8950 4200
+Wire Wire Line
+	10350 4000 10350 4200
+Wire Wire Line
+	9400 4200 8950 4200
+Connection ~ 8950 4200
+Wire Wire Line
+	8950 4200 8950 4700
+Wire Wire Line
+	9700 4200 10350 4200
+Connection ~ 10350 4200
+Wire Wire Line
+	10350 4200 10350 4700
 $EndSCHEMATC
