File: pcb_1/pcb_1.sch (KiCad schematic (older format))
At the start: 50 parts, among them J1 Screw_Terminal_01x02, J2 Screw_Terminal_01x03, J3 Conn_Relay, J4 Screw_Terminal_01x02, K1 DIPxx-1Axx-11x, Q1 BD139, Q7 Q_NMOS_DGS, U1 MAX9944, U2 SPX2920U-5.0, U3 INA240A1PWR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

Commit message: pcb: Kaikki vedot tehty
Parts:
- C2: footprint Capacitors_THT:CP_Radial_D8.0mm_P5.00mm -> Capacitors_SMD:C_1206_HandSoldering; symbol Device:CP -> Device:C
- C6, C8: value C -> 10u; footprint Capacitors_SMD:C_0805_HandSoldering -> Capacitors_SMD:C_1206_HandSoldering
- Rs1: footprint Resistors_SMD:R_2816 -> Resistors_SMD:R_2512_HandSoldering
Changed lines of the file:
@@
 F 0 "Rs1" V 8280 3800 50  0000 C CNN
 F 1 "0.1" V 8200 3800 50  0000 C CNN
-F 2 "Resistors_SMD:R_2816" V 8130 3800 50  0001 C CNN
+F 2 "Resistors_SMD:R_2512_HandSoldering" V 8130 3800 50  0001 C CNN
 F 3 "" H 8200 3800 50  0000 C CNN
 	1    8200 3800
@@
 $Comp
 L lab_power_supply:MAX9944 U1
-U 1 1 5DD19535
+U 2 1 5DD19535
 P 6650 1750
 F 0 "U1" H 6750 2050 50  0000 C CNN
@@
 F 2 "Housings_SOIC:SOIC-8_3.9x4.9mm_Pitch1.27mm" H 6650 1750 50  0001 C CNN
 F 3 "http://www.ti.com/lit/ds/symlink/lm358.pdf" H 6650 1750 50  0001 C CNN
-	1    6650 1750
+	2    6650 1750
 	1    0    0    -1
 $EndComp
@@
 $EndComp
 $Comp
-L Device:CP C2
+L Device:C C2
 U 1 1 5DD2D3D7
 P 4700 2050
 F 0 "C2" H 4750 2150 50  0000 L CNN
 F 1 "10u" H 4750 1950 50  0000 L CNN
-F 2 "Capacitors_THT:CP_Radial_D8.0mm_P5.00mm" H 4738 1900 50  0001 C CNN
+F 2 "Capacitors_SMD:C_1206_HandSoldering" H 4738 1900 50  0001 C CNN
 F 3 "~" H 4700 2050 50  0001 C CNN
 	1    4700 2050
@@
 $Comp
 L lab_power_supply:MAX9944 U1
-U 2 1 5DD2E469
+U 1 1 5DD2E469
 P 6650 2600
 F 0 "U1" H 6750 2900 50  0000 C CNN
@@
 F 2 "Housings_SOIC:SOIC-8_3.9x4.9mm_Pitch1.27mm" H 6650 2600 50  0001 C CNN
 F 3 "http://www.ti.com/lit/ds/symlink/lm358.pdf" H 6650 2600 50  0001 C CNN
-	2    6650 2600
+	1    6650 2600
 	1    0    0    -1
 $EndComp
@@
 	0    1    1    0
 $EndComp
+Text GLabel 3650 6400 2    60   Input ~ 0
+Iset
 Text GLabel 3650 6200 2    60   Input ~ 0
-Iset
-Text GLabel 3650 6400 2    60   Input ~ 0
 Vset
 Wire Wire Line
@@
 P 5450 5150
 F 0 "C8" V 5198 5150 50  0000 C CNN
-F 1 "C" V 5289 5150 50  0000 C CNN
-F 2 "Capacitors_SMD:C_0805_HandSoldering" H 5488 5000 50  0001 C CNN
+F 1 "10u" V 5289 5150 50  0000 C CNN
+F 2 "Capacitors_SMD:C_1206_HandSoldering" H 5488 5000 50  0001 C CNN
 F 3 "~" H 5450 5150 50  0001 C CNN
 	1    5450 5150
@@
 P 4900 3450
 F 0 "C6" H 5015 3496 50  0000 L CNN
-F 1 "C" H 5015 3405 50  0000 L CNN
-F 2 "Capacitors_SMD:C_0805_HandSoldering" H 4938 3300 50  0001 C CNN
+F 1 "10u" H 5015 3405 50  0000 L CNN
+F 2 "Capacitors_SMD:C_1206_HandSoldering" H 4938 3300 50  0001 C CNN
 F 3 "~" H 4900 3450 50  0001 C CNN
 	1    4900 3450

Commit message: Toinen konkka lisätty
Parts:
- added C18: CP, Capacitors_THT:CP_Radial_D30.0mm_P10.00mm_SnapIn, symbol Device:CP
Connections:
- wire segments 170 -> 171
Changed lines of the file:
@@
 Connection ~ 5250 1750
 Wire Wire Line
-	4000 1200 5250 1200
+	4000 1200 4750 1200
 Connection ~ 5250 1200
 $Comp
@@
 Wire Wire Line
 	10350 4200 10350 4700
+$Comp
+L Device:CP C18
+U 1 1 5DD2774F
+P 4750 1350
+F 0 "C18" H 4868 1396 50  0000 L CNN
+F 1 "CP" H 4868 1305 50  0000 L CNN
+F 2 "Capacitors_THT:CP_Radial_D30.0mm_P10.00mm_SnapIn" H 4788 1200 50  0001 C CNN
+F 3 "~" H 4750 1350 50  0001 C CNN
+	1    4750 1350
+	1    0    0    -1
+$EndComp
+Connection ~ 4750 1200
+Wire Wire Line
+	4750 1200 5250 1200
+$Comp
+L power:GNDA #PWR0102
+U 1 1 5DD2892C
+P 4750 1500
+F 0 "#PWR0102" H 4750 1250 50  0001 C CNN
+F 1 "GNDA" H 4755 1327 50  0000 C CNN
+F 2 "" H 4750 1500 50  0001 C CNN
+F 3 "" H 4750 1500 50  0001 C CNN
+	1    4750 1500
+	1    0    0    -1
+$EndComp
 $EndSCHEMATC

Commit message: pcb: Suodatuskonkat ja kiinnitysreiät lisätty
Parts:
- added C19: CP, Capacitors_THT:CP_Radial_D8.0mm_P5.00mm, symbol Device:CP
- added C20: C, Capacitors_THT:C_Disc_D7.5mm_W5.0mm_P5.00mm, symbol Device:C
- C1: renamed from C18; value CP -> 4700u
- C2: renamed from CP1; value 15000uF 50V -> 15000u
- renumbered C1 to C18, C2 to C21, Cb1 to C22, Cb2 to C23, Cb3 to C24, Cb4 to C25
Connections:
- wire segments 171 -> 176
Other:
- moved on the sheet: C1, C2, C21, C3, D3

Commit message: NMOS-symbolit muutettu
Parts:
- removed Q7: Q_NMOS_DGS, TO_SOT_Packages_SMD:SuperSOT-3, symbol Device:Q_NMOS_DGS
- added Q7: Q_NMOS_GSD, TO_SOT_Packages_SMD:SuperSOT-3, symbol Device:Q_NMOS_GSD
Changed lines of the file:
@@
 Wire Wire Line
 	8500 2400 8200 2400
-$Comp
-L Device:Q_NMOS_DGS Q7
-U 1 1 5DD62A9A
-P 10250 3800
-F 0 "Q7" H 10456 3754 50  0000 L CNN
-F 1 "Q_NMOS_DGS" H 10456 3845 50  0000 L CNN
-F 2 "TO_SOT_Packages_SMD:SuperSOT-3" H 10450 3900 50  0001 C CNN
-F 3 "~" H 10250 3800 50  0001 C CNN
-	1    10250 3800
-	1    0    0    1
-$EndComp
 Wire Wire Line
 	10350 4700 9850 4700
@@
 Wire Wire Line
 	3750 1200 4400 1200
+$Comp
+L Device:Q_NMOS_GSD Q7
+U 1 1 5DD8B0EF
+P 10250 3800
+F 0 "Q7" H 10456 3754 50  0000 L CNN
+F 1 "Q_NMOS_GSD" H 10456 3845 50  0000 L CNN
+F 2 "TO_SOT_Packages_SMD:SuperSOT-3" H 10450 3900 50  0001 C CNN
+F 3 "~" H 10250 3800 50  0001 C CNN
+	1    10250 3800
+	1    0    0    1
+$EndComp
 $EndSCHEMATC

Commit message: pcb: Silkscreeniä päivitetty
Parts:
- C7: footprint Capacitors_THT:CP_Radial_D8.0mm_P5.00mm -> Capacitor_THT:CP_Radial_D6.3mm_P2.50mm
Changed lines of the file:
@@
 F 0 "C7" H 5418 3496 50  0000 L CNN
 F 1 "100u" H 5418 3405 50  0000 L CNN
-F 2 "Capacitors_THT:CP_Radial_D8.0mm_P5.00mm" H 5338 3300 50  0001 C CNN
+F 2 "Capacitor_THT:CP_Radial_D6.3mm_P2.50mm" H 5338 3300 50  0001 C CNN
 F 3 "~" H 5300 3450 50  0001 C CNN
 	1    5300 3450

Commit message: pcb: Kondensaattoreiden footprintit muuttettu
Parts:
- C10, C11, C18, C22, C23, C24, C25, C3, C4, C5, C9: footprint Capacitors_SMD:C_0805_HandSoldering -> Capacitor_SMD:C_0805_2012Metric_Pad1.15x1.40mm_HandSolder
- C21, C8: footprint Capacitors_SMD:C_1206_HandSoldering -> Capacitor_SMD:C_0805_2012Metric_Pad1.15x1.40mm_HandSolder
- C6: footprint Capacitors_SMD:C_1206_HandSoldering -> Capacitor_SMD:C_0603_1608Metric_Pad1.05x0.95mm_HandSolder
Changed lines of the file:
@@
 F 0 "C24" H 2475 6900 50  0000 L CNN
 F 1 "0.1u" H 2475 6700 50  0000 L CNN
-F 2 "Capacitors_SMD:C_0805_HandSoldering" H 2488 6650 50  0001 C CNN
+F 2 "Capacitor_SMD:C_0805_2012Metric_Pad1.15x1.40mm_HandSolder" H 2488 6650 50  0001 C CNN
 F 3 "" H 2450 6800 50  0000 C CNN
 	1    2450 6800
@@
 F 0 "C23" V 1950 5350 50  0000 L CNN
 F 1 "0.1u" V 1850 5350 50  0000 L CNN
-F 2 "Capacitors_SMD:C_0805_HandSoldering" H 1738 5300 50  0001 C CNN
+F 2 "Capacitor_SMD:C_0805_2012Metric_Pad1.15x1.40mm_HandSolder" H 1738 5300 50  0001 C CNN
 F 3 "" H 1700 5450 50  0000 C CNN
 	1    1700 5450
@@
 F 0 "C22" H 4575 3550 50  0000 L CNN
 F 1 "0.1u" H 4575 3350 50  0000 L CNN
-F 2 "Capacitors_SMD:C_0805_HandSoldering" H 4588 3300 50  0001 C CNN
+F 2 "Capacitor_SMD:C_0805_2012Metric_Pad1.15x1.40mm_HandSolder" H 4588 3300 50  0001 C CNN
 F 3 "" H 4550 3450 50  0000 C CNN
 	1    4550 3450
@@
 F 0 "C25" H 2450 6900 50  0000 L CNN
 F 1 "0.1u" H 2450 6700 50  0000 L CNN
-F 2 "Capacitors_SMD:C_0805_HandSoldering" H 2688 6650 50  0001 C CNN
+F 2 "Capacitor_SMD:C_0805_2012Metric_Pad1.15x1.40mm_HandSolder" H 2688 6650 50  0001 C CNN
 F 3 "" H 2650 6800 50  0000 C CNN
 	1    2650 6800
@@
 F 0 "C18" V 6600 2100 50  0000 C CNN
 F 1 "C" V 6600 1900 50  0000 C CNN
-F 2 "Capacitors_SMD:C_0805_HandSoldering" H 6688 1850 50  0001 C CNN
+F 2 "Capacitor_SMD:C_0805_2012Metric_Pad1.15x1.40mm_HandSolder" H 6688 1850 50  0001 C CNN
 F 3 "~" H 6650 2000 50  0001 C CNN
 	1    6650 2000
@@
 F 0 "C3" H 5050 2450 50  0000 L CNN
 F 1 "0.1u" H 5050 2250 50  0000 L CNN
-F 2 "Capacitors_SMD:C_0805_HandSoldering" H 5038 2200 50  0001 C CNN
+F 2 "Capacitor_SMD:C_0805_2012Metric_Pad1.15x1.40mm_HandSolder" H 5038 2200 50  0001 C CNN
 F 3 "~" H 5000 2350 50  0001 C CNN
 	1    5000 2350
@@
 F 0 "C21" H 4750 2450 50  0000 L CNN
 F 1 "10u" H 4750 2250 50  0000 L CNN
-F 2 "Capacitors_SMD:C_1206_HandSoldering" H 4738 2200 50  0001 C CNN
+F 2 "Capacitor_SMD:C_0805_2012Metric_Pad1.15x1.40mm_HandSolder" H 4738 2200 50  0001 C CNN
 F 3 "~" H 4700 2350 50  0001 C CNN
 	1    4700 2350
@@
 F 0 "C9" V 5300 5400 50  0000 C CNN
 F 1 "0.1u" V 5200 5350 50  0000 C CNN
-F 2 "Capacitors_SMD:C_0805_HandSoldering" H 5488 5250 50  0001 C CNN
+F 2 "Capacitor_SMD:C_0805_2012Metric_Pad1.15x1.40mm_HandSolder" H 5488 5250 50  0001 C CNN
 F 3 "~" H 5450 5400 50  0001 C CNN
 	1    5450 5400
@@
 F 0 "C4" V 6700 2750 50  0000 C CNN
 F 1 "C" V 6700 2950 50  0000 C CNN
-F 2 "Capacitors_SMD:C_0805_HandSoldering" H 6688 2700 50  0001 C CNN
+F 2 "Capacitor_SMD:C_0805_2012Metric_Pad1.15x1.40mm_HandSolder" H 6688 2700 50  0001 C CNN
 F 3 "~" H 6650 2850 50  0001 C CNN
 	1    6650 2850
@@
 F 0 "C11" H 3285 6504 50  0000 R CNN
 F 1 "0.1u" H 3285 6595 50  0000 R CNN
-F 2 "Capacitors_SMD:C_0805_HandSoldering" H 3438 6400 50  0001 C CNN
+F 2 "Capacitor_SMD:C_0805_2012Metric_Pad1.15x1.40mm_HandSolder" H 3438 6400 50  0001 C CNN
 F 3 "~" H 3400 6550 50  0001 C CNN
 	1    3400 6550
@@
 F 0 "C10" H 3515 6096 50  0000 L CNN
 F 1 "0.1u" H 3515 6005 50  0000 L CNN
-F 2 "Capacitors_SMD:C_0805_HandSoldering" H 3438 5900 50  0001 C CNN
+F 2 "Capacitor_SMD:C_0805_2012Metric_Pad1.15x1.40mm_HandSolder" H 3438 5900 50  0001 C CNN
 F 3 "~" H 3400 6050 50  0001 C CNN
 	1    3400 6050
@@
 F 0 "C5" H 3350 3500 50  0000 L CNN
 F 1 "0.22u" H 3200 3400 50  0000 L CNN
-F 2 "Capacitors_SMD:C_0805_HandSoldering" H 3588 3300 50  0001 C CNN
+F 2 "Capacitor_SMD:C_0805_2012Metric_Pad1.15x1.40mm_HandSolder" H 3588 3300 50  0001 C CNN
 F 3 "~" H 3550 3450 50  0001 C CNN
 	1    3550 3450
@@
 F 0 "C8" V 5198 5150 50  0000 C CNN
 F 1 "10u" V 5289 5150 50  0000 C CNN
-F 2 "Capacitors_SMD:C_1206_HandSoldering" H 5488 5000 50  0001 C CNN
+F 2 "Capacitor_SMD:C_0805_2012Metric_Pad1.15x1.40mm_HandSolder" H 5488 5000 50  0001 C CNN
 F 3 "~" H 5450 5150 50  0001 C CNN
 	1    5450 5150
@@
 F 0 "C6" H 5015 3496 50  0000 L CNN
 F 1 "10u" H 5015 3405 50  0000 L CNN
-F 2 "Capacitors_SMD:C_1206_HandSoldering" H 4938 3300 50  0001 C CNN
+F 2 "Capacitor_SMD:C_0603_1608Metric_Pad1.05x0.95mm_HandSolder" H 4938 3300 50  0001 C CNN
 F 3 "~" H 4900 3450 50  0001 C CNN
 	1    4900 3450
