File: pcb_1/Micrcontroller.sch (KiCad schematic (older format))
At the start: 24 parts, among them J4 AVR-ISP-6, J5 AVR-ISP-6, Q2 Q_PMOS_DGS, Q3 Q_PMOS_DGS, Q4 Q_PMOS_DGS, Q5 Q_PMOS_DGS, U10 HCPL2601SD, U11 HCPL2601SD, U4 ATmega328PB-AU, U8 HCPL2631SD

Commit message: pcb: Add relay and filtering capacitors
Parts:
- removed C8: 0.1u, symbol Device:C
- removed J5: AVR-ISP-6, symbol Connector:AVR-ISP-6
- removed Q5: Q_PMOS_DGS, symbol Device:Q_PMOS_DGS
- removed R17: 330, symbol Device:R
- removed U10: HCPL2601SD, symbol lab_power_supply:HCPL2601SD
- added C?: 0.1u, symbol Device:C
- added J: Isolated_ISP, symbol lab_power_supply:Isolated_ISP
- added Q? (x2): Q_PMOS_DGS, symbol Device:Q_PMOS_DGS
- added R? (x2): 330, symbol Device:R
- added R?: 10k, symbol Device:R
- added U?: HCPL2631SD, symbol lab_power_supply:HCPL2631SD
Connections:
- net labels added: SLAVE_RESET, UNREG_MON
- wire segments 108 -> 121
- no-connect marks 1 -> 2
Other:
- moved on the sheet: C9, R11, R14, R5

Commit message: pcb: Fix mismatching global labels
Also add connections for thermistors.
Parts:
- added J7: THERM0, symbol Connector_Generic:Conn_02x01
- added J8: THERM1, symbol Connector_Generic:Conn_02x01
- added R16: 100, symbol Device:R
- added R18, R19: R, symbol Device:R
- Q2: renamed from Q3; value Q_PMOS_DGS -> Q_NMOS_DGS; symbol Device:Q_PMOS_DGS -> Device:Q_NMOS_DGS
- Q3: renamed from Q4; value Q_PMOS_DGS -> Q_NMOS_DGS; symbol Device:Q_PMOS_DGS -> Device:Q_NMOS_DGS
- Q4, Q5: renamed from Q?; value Q_PMOS_DGS -> Q_NMOS_DGS; symbol Device:Q_PMOS_DGS -> Device:Q_NMOS_DGS
- Q6: renamed from Q2; value Q_PMOS_DGS -> Q_NMOS_DGS; symbol Device:Q_PMOS_DGS -> Device:Q_NMOS_DGS
- gave numbers to parts that had none: 5
- renumbered C7 to C10, C5 to C12, C6 to C13, C9 to C14, J to J5, J4 to J6, R16 to R10, R10 to R13, R12 to R14, R13 to R15, R14 to R17, R11 to R20, R5 to R21, R15 to R9, U8 to U6, U11 to U8, U4 to U9
Connections:
- net labels added: DAC_LDAC, DAC_SDI
- net labels removed: DAC_MOSI
- wire segments 121 -> 132
- no-connect marks 2 -> 15
Other:
- moved on the sheet: R20, R21

Commit message: pcb: Add Zener regulator to op-amp supply
Parts:
- added C16: 0.1u, symbol Device:C
- renumbered C10 to C12, C11 to C13, C12 to C14, C13 to C15, C14 to C17, R9 to R10, R10 to R11, R11 to R12, R12 to R13, R13 to R14, R14 to R15, R15 to R16, R16 to R17, R17 to R18, R18 to R19, R19 to R20, R20 to R21, R21 to R22, R22 to R23
Connections:
- wire segments 132 -> 134
- no-connect marks 15 -> 14
Changed lines of the file:
@@
 EESchema Schematic File Version 4
+LIBS:pcb_1-cache
 EELAYER 30 0
 EELAYER END
@@
 $EndDescr
 $Comp
-L power:GNDD #PWR034
+L power:GNDD #PWR036
 U 1 1 5DD60E95
 P 2600 6800
-F 0 "#PWR034" H 2600 6550 50  0001 C CNN
+F 0 "#PWR036" H 2600 6550 50  0001 C CNN
 F 1 "GNDD" H 2604 6645 50  0000 C CNN
 F 2 "" H 2600 6800 50  0001 C CNN
@@
 $EndComp
 $Comp
-L Device:C C12
+L Device:C C14
 U 1 1 5DD639F1
 P 2400 3700
-F 0 "C12" V 2148 3700 50  0000 C CNN
+F 0 "C14" V 2148 3700 50  0000 C CNN
 F 1 "0.1u" V 2239 3700 50  0000 C CNN
 F 2 "" H 2438 3550 50  0001 C CNN
@@
 $EndComp
 $Comp
-L power:+5V #PWR023
+L power:+5V #PWR025
 U 1 1 5DD6BCEE
 P 5100 4800
-F 0 "#PWR023" H 5100 4650 50  0001 C CNN
+F 0 "#PWR025" H 5100 4650 50  0001 C CNN
 F 1 "+5V" H 5115 4973 50  0000 C CNN
 F 2 "" H 5100 4800 50  0001 C CNN
@@
 $EndComp
 $Comp
-L Device:R R21
+L Device:R R22
 U 1 1 5DD6F284
 P 1900 5600
-F 0 "R21" H 1970 5646 50  0000 L CNN
+F 0 "R22" H 1970 5646 50  0000 L CNN
 F 1 "5k" H 1970 5555 50  0000 L CNN
 F 2 "" V 1830 5600 50  0001 C CNN
@@
 $EndComp
 $Comp
-L Device:R R20
+L Device:R R21
 U 1 1 5DD6F85B
 P 1650 5600
-F 0 "R20" H 1720 5646 50  0000 L CNN
+F 0 "R21" H 1720 5646 50  0000 L CNN
 F 1 "5k" H 1720 5555 50  0000 L CNN
 F 2 "" V 1580 5600 50  0001 C CNN
@@
 	3500 4300 4300 4300
 $Comp
-L Device:R R13
+L Device:R R14
 U 1 1 5DD7ACAD
 P 3800 3900
-F 0 "R13" H 3870 3946 50  0000 L CNN
+F 0 "R14" H 3870 3946 50  0000 L CNN
 F 1 "100" H 3870 3855 50  0000 L CNN
 F 2 "" V 3730 3900 50  0001 C CNN
@@
 $EndComp
 $Comp
-L Device:R R15
+L Device:R R16
 U 1 1 5DD7B76E
 P 4300 3900
-F 0 "R15" H 4370 3946 50  0000 L CNN
+F 0 "R16" H 4370 3946 50  0000 L CNN
 F 1 "100" H 4370 3855 50  0000 L CNN
 F 2 "" V 4230 3900 50  0001 C CNN
@@
 $EndComp
 $Comp
-L Device:R R14
+L Device:R R15
 U 1 1 5DD7B4E3
 P 4050 3900
-F 0 "R14" H 4120 3946 50  0000 L CNN
+F 0 "R15" H 4120 3946 50  0000 L CNN
 F 1 "100" H 4120 3855 50  0000 L CNN
 F 2 "" V 3980 3900 50  0001 C CNN
@@
 $EndComp
 $Comp
-L Device:R R9
+L Device:R R10
 U 1 1 5DDEC927
 P 9000 900
-F 0 "R9" V 8950 1050 50  0000 C CNN
+F 0 "R10" V 8950 1050 50  0000 C CNN
 F 1 "330" V 9050 1100 50  0000 C CNN
 F 2 "" V 8930 900 50  0001 C CNN
@@
 $EndComp
 $Comp
-L Device:R R10
+L Device:R R11
 U 1 1 5DDF29FD
 P 9000 1650
-F 0 "R10" V 8950 1800 50  0000 C CNN
+F 0 "R11" V 8950 1800 50  0000 C CNN
 F 1 "330" V 9050 1850 50  0000 C CNN
 F 2 "" V 8930 1650 50  0001 C CNN
@@
 $EndComp
 $Comp
-L power:GNDD #PWR024
+L power:GNDD #PWR026
 U 1 1 5DE46C99
 P 8800 4900
-F 0 "#PWR024" H 8800 4650 50  0001 C CNN
+F 0 "#PWR026" H 8800 4650 50  0001 C CNN
 F 1 "GNDD" V 8804 4790 50  0000 R CNN
 F 2 "" H 8800 4900 50  0001 C CNN
@@
 	8050 4800 8800 4800
 $Comp
-L power:GNDD #PWR027
+L power:GNDD #PWR029
 U 1 1 5DE4D380
 P 9900 5100
-F 0 "#PWR027" H 9900 4850 50  0001 C CNN
+F 0 "#PWR029" H 9900 4850 50  0001 C CNN
 F 1 "GNDD" H 9904 4945 50  0000 C CNN
 F 2 "" H 9900 5100 50  0001 C CNN
@@
 $EndComp
 $Comp
-L Device:C C14
+L Device:C C17
 U 1 1 5DE4EB0D
 P 9900 4850
-F 0 "C14" H 9785 4804 50  0000 R CNN
+F 0 "C17" H 9785 4804 50  0000 R CNN
 F 1 "0.1u" H 9785 4895 50  0000 R CNN
 F 2 "" H 9938 4700 50  0001 C CNN
@@
 	9650 5000 9900 5000
 $Comp
-L power:GNDD #PWR028
+L power:GNDD #PWR030
 U 1 1 5DE61505
 P 8050 5350
-F 0 "#PWR028" H 8050 5100 50  0001 C CNN
+F 0 "#PWR030" H 8050 5100 50  0001 C CNN
 F 1 "GNDD" H 8054 5195 50  0000 C CNN
 F 2 "" H 8050 5350 50  0001 C CNN
@@
 	8050 4800 8050 4850
 $Comp
-L Device:R R17
+L Device:R R18
 U 1 1 5DE6A4FF
 P 8050 4650
-F 0 "R17" H 8120 4696 50  0000 L CNN
+F 0 "R18" H 8120 4696 50  0000 L CNN
 F 1 "500" H 8120 4605 50  0000 L CNN
 F 2 "" V 7980 4650 50  0001 C CNN
@@
 Connection ~ 8050 4800
 $Comp
-L power:+5V #PWR022
+L power:+5V #PWR023
 U 1 1 5DE6B0EB
 P 8050 4500
-F 0 "#PWR022" H 8050 4350 50  0001 C CNN
+F 0 "#PWR023" H 8050 4350 50  0001 C CNN
 F 1 "+5V" H 8065 4673 50  0000 C CNN
 F 2 "" H 8050 4500 50  0001 C CNN
@@
 	9650 4900 9750 4900
 $Comp
-L Device:C C10
+L Device:C C12
 U 1 1 5DE807E4
 P 5800 1750
-F 0 "C10" H 6000 1700 50  0000 R CNN
+F 0 "C12" H 6000 1700 50  0000 R CNN
 F 1 "0.1u" H 6050 1800 50  0000 R CNN
 F 2 "" H 5838 1600 50  0001 C CNN
@@
 	2700 3700 2600 3700
 $Comp
-L Device:C C13
+L Device:C C15
 U 1 1 5DEC2D6D
 P 2850 3700
-F 0 "C13" V 2598 3700 50  0000 C CNN
+F 0 "C15" V 2598 3700 50  0000 C CNN
 F 1 "C" V 2689 3700 50  0000 C CNN
 F 2 "" H 2888 3550 50  0001 C CNN
@@
 	0    -1   -1   0
 $EndComp
-NoConn ~ 2000 4100
 Wire Wire Line
 	3200 5100 3450 5100
@@
 Connection ~ 1650 5800
 $Comp
-L power:+5V #PWR030
+L power:+5V #PWR032
 U 1 1 5DD01499
 P 1900 5450
-F 0 "#PWR030" H 1900 5300 50  0001 C CNN
+F 0 "#PWR032" H 1900 5300 50  0001 C CNN
 F 1 "+5V" H 1915 5623 50  0000 C CNN
 F 2 "" H 1900 5450 50  0001 C CNN
@@
 $EndComp
 $Comp
-L power:+5V #PWR029
+L power:+5V #PWR031
 U 1 1 5DD01A9D
 P 1650 5450
-F 0 "#PWR029" H 1650 5300 50  0001 C CNN
+F 0 "#PWR031" H 1650 5300 50  0001 C CNN
 F 1 "+5V" H 1665 5623 50  0000 C CNN
 F 2 "" H 1650 5450 50  0001 C CNN
@@
 $EndComp
 $Comp
-L Device:R R11
+L Device:R R12
 U 1 1 5DDA6759
 P 9000 2400
-F 0 "R11" V 8950 2550 50  0000 C CNN
+F 0 "R12" V 8950 2550 50  0000 C CNN
 F 1 "330" V 9050 2600 50  0000 C CNN
 F 2 "" V 8930 2400 50  0001 C CNN
@@
 $EndComp
 $Comp
-L Device:R R12
+L Device:R R13
 U 1 1 5DDA676E
 P 9000 3150
-F 0 "R12" V 8950 3300 50  0000 C CNN
+F 0 "R13" V 8950 3300 50  0000 C CNN
 F 1 "330" V 9050 3350 50  0000 C CNN
 F 2 "" V 8930 3150 50  0001 C CNN
@@
 Connection ~ 8850 2400
 $Comp
-L Device:C C11
+L Device:C C13
 U 1 1 5DDA6796
 P 5800 3250
-F 0 "C11" H 6000 3200 50  0000 R CNN
+F 0 "C13" H 6000 3200 50  0000 R CNN
 F 1 "0.1u" H 6050 3300 50  0000 R CNN
 F 2 "" H 5838 3100 50  0001 C CNN
@@
 	9750 1500 10050 1500
 $Comp
-L Device:R R22
+L Device:R R23
 U 1 1 5DE001F9
 P 3400 5750
-F 0 "R22" H 3330 5704 50  0000 R CNN
+F 0 "R23" H 3330 5704 50  0000 R CNN
 F 1 "10k" H 3330 5795 50  0000 R CNN
 F 2 "" V 3330 5750 50  0001 C CNN
@@
 Connection ~ 3400 5600
 $Comp
-L power:+5V #PWR031
+L power:+5V #PWR033
 U 1 1 5DE019EC
 P 3400 5900
-F 0 "#PWR031" H 3400 5750 50  0001 C CNN
+F 0 "#PWR033" H 3400 5750 50  0001 C CNN
 F 1 "+5V" H 3415 6073 50  0000 C CNN
 F 2 "" H 3400 5900 50  0001 C CNN
@@
 Wire Wire Line
 	2000 5800 1650 5800
-$Comp
-L MCU_Microchip_ATmega:ATmega328PB-AU U9
-U 1 1 5DD5F79A
-P 2600 5300
-F 0 "U9" H 2000 3700 50  0000 C CNN
-F 1 "ATmega328PB-AU" H 2000 3800 50  0000 C CNN
-F 2 "Package_QFP:TQFP-32_7x7mm_P0.8mm" H 2600 5300 50  0001 C CIN
-F 3 "http://ww1.microchip.com/downloads/en/DeviceDoc/40001906C.pdf" H 2600 5300 50  0001 C CNN
-	1    2600 5300
-	1    0    0    -1
-$EndComp
 Wire Wire Line
 	1500 6000 2000 6000
 $Comp
-L power:+5V #PWR025
+L power:+5V #PWR027
 U 1 1 5DD419C2
 P 4200 5050
-F 0 "#PWR025" H 4200 4900 50  0001 C CNN
+F 0 "#PWR027" H 4200 4900 50  0001 C CNN
 F 1 "+5V" H 4215 5223 50  0000 C CNN
 F 2 "" H 4200 5050 50  0001 C CNN
@@
 $EndComp
 $Comp
-L power:+5V #PWR026
+L power:+5V #PWR028
 U 1 1 5DD42300
 P 4450 5050
-F 0 "#PWR026" H 4450 4900 50  0001 C CNN
+F 0 "#PWR028" H 4450 4900 50  0001 C CNN
 F 1 "+5V" H 4465 5223 50  0000 C CNN
 F 2 "" H 4450 5050 50  0001 C CNN
@@
 $EndComp
 $Comp
-L power:GNDD #PWR033
+L power:GNDD #PWR035
 U 1 1 5DD42F65
 P 4450 6050
-F 0 "#PWR033" H 4450 5800 50  0001 C CNN
+F 0 "#PWR035" H 4450 5800 50  0001 C CNN
 F 1 "GNDD" H 4454 5895 50  0000 C CNN
 F 2 "" H 4450 6050 50  0001 C CNN
@@
 $EndComp
 $Comp
-L power:GNDD #PWR032
+L power:GNDD #PWR034
 U 1 1 5DD4257C
 P 4200 6050
-F 0 "#PWR032" H 4200 5800 50  0001 C CNN
+F 0 "#PWR034" H 4200 5800 50  0001 C CNN
 F 1 "GNDD" H 4204 5895 50  0000 C CNN
 F 2 "" H 4200 6050 50  0001 C CNN
@@
 	4200 5350 4200 5400
 $Comp
-L Device:R R18
+L Device:R R19
 U 1 1 5DD26697
 P 4200 5200
-F 0 "R18" H 4270 5246 50  0000 L CNN
+F 0 "R19" H 4270 5246 50  0000 L CNN
 F 1 "R" H 4270 5155 50  0000 L CNN
 F 2 "" V 4130 5200 50  0001 C CNN
@@
 $EndComp
 $Comp
-L Device:R R19
+L Device:R R20
 U 1 1 5DD25C52
 P 4450 5200
-F 0 "R19" H 4520 5246 50  0000 L CNN
+F 0 "R20" H 4520 5246 50  0000 L CNN
 F 1 "R" H 4520 5155 50  0000 L CNN
 F 2 "" V 4380 5200 50  0001 C CNN
@@
 SLAVE_RESET
 $Comp
-L Device:R R16
+L Device:R R17
 U 1 1 5DE51582
 P 4550 3900
-F 0 "R16" H 4620 3946 50  0000 L CNN
+F 0 "R17" H 4620 3946 50  0000 L CNN
 F 1 "100" H 4620 3855 50  0000 L CNN
 F 2 "" V 4480 3900 50  0001 C CNN
@@
 $EndComp
 $Comp
-L power:+5V #PWR0101
+L power:+5V #PWR024
 U 1 1 5DE715DD
 P 9900 4650
-F 0 "#PWR0101" H 9900 4500 50  0001 C CNN
+F 0 "#PWR024" H 9900 4500 50  0001 C CNN
 F 1 "+5V" H 9915 4823 50  0000 C CNN
 F 2 "" H 9900 4650 50  0001 C CNN
@@
 Wire Wire Line
 	9900 4650 9900 4700
+$Comp
+L Device:C C16
+U 1 1 5DD76A41
+P 1900 4300
+F 0 "C16" H 1700 4350 50  0000 L CNN
+F 1 "0.1u" H 1600 4250 50  0000 L CNN
+F 2 "" H 1938 4150 50  0001 C CNN
+F 3 "~" H 1900 4300 50  0001 C CNN
+	1    1900 4300
+	1    0    0    -1
+$EndComp
+Wire Wire Line
+	1900 4150 1900 4100
+Wire Wire Line
+	1900 4100 2000 4100
+$Comp
+L MCU_Microchip_ATmega:ATmega328PB-AU U9
+U 1 1 5DD5F79A
+P 2600 5300
+F 0 "U9" H 2000 3700 50  0000 C CNN
+F 1 "ATmega328PB-AU" H 2000 3800 50  0000 C CNN
+F 2 "Package_QFP:TQFP-32_7x7mm_P0.8mm" H 2600 5300 50  0001 C CIN
+F 3 "http://ww1.microchip.com/downloads/en/DeviceDoc/40001906C.pdf" H 2600 5300 50  0001 C CNN
+	1    2600 5300
+	1    0    0    -1
+$EndComp
+$Comp
+L power:GNDD #PWR022
+U 1 1 5DD7F113
+P 1900 4450
+F 0 "#PWR022" H 1900 4200 50  0001 C CNN
+F 1 "GNDD" H 1904 4295 50  0000 C CNN
+F 2 "" H 1900 4450 50  0001 C CNN
+F 3 "" H 1900 4450 50  0001 C CNN
+	1    1900 4450
+	1    0    0    -1
+$EndComp
 $EndSCHEMATC

Commit message: Footprintit lisätty ja pcb-layout aloitettu
Parts:
- C12, C13, C14, C15, C16, C17: footprint (none) -> Capacitors_SMD:C_0805_HandSoldering
- J5: footprint (none) -> Pin_Headers:Pin_Header_Straight_1x08_Pitch2.54mm
- J6: footprint (none) -> Pin_Headers:Pin_Header_Straight_2x03_Pitch2.54mm
- J7, J8: footprint (none) -> Pin_Headers:Pin_Header_Straight_1x02_Pitch2.54mm
- Q2, Q3, Q4, Q5, Q6: footprint (none) -> TO_SOT_Packages_SMD:SuperSOT-3
- R10, R11, R12, R13, R14, R15, R16, R17, R18, R19, R20, R21, R22, R23: footprint (none) -> Resistors_SMD:R_0805_HandSoldering
- U6, U7, U8: footprint (none) -> lab_power_supply:HCPL2631SD
- U9: footprint Package_QFP:TQFP-32_7x7mm_P0.8mm -> Housings_QFP:TQFP-32_7x7mm_Pitch0.8mm
Changed lines of the file:
@@
 EESchema Schematic File Version 4
-LIBS:pcb_1-cache
 EELAYER 30 0
 EELAYER END
@@
 F 0 "C14" V 2148 3700 50  0000 C CNN
 F 1 "0.1u" V 2239 3700 50  0000 C CNN
-F 2 "" H 2438 3550 50  0001 C CNN
+F 2 "Capacitors_SMD:C_0805_HandSoldering" H 2438 3550 50  0001 C CNN
 F 3 "~" H 2400 3700 50  0001 C CNN
 	1    2400 3700
@@
 F 0 "R22" H 1970 5646 50  0000 L CNN
 F 1 "5k" H 1970 5555 50  0000 L CNN
-F 2 "" V 1830 5600 50  0001 C CNN
+F 2 "Resistors_SMD:R_0805_HandSoldering" V 1830 5600 50  0001 C CNN
 F 3 "~" H 1900 5600 50  0001 C CNN
 	1    1900 5600
@@
 F 0 "R21" H 1720 5646 50  0000 L CNN
 F 1 "5k" H 1720 5555 50  0000 L CNN
-F 2 "" V 1580 5600 50  0001 C CNN
+F 2 "Resistors_SMD:R_0805_HandSoldering" V 1580 5600 50  0001 C CNN
 F 3 "~" H 1650 5600 50  0001 C CNN
 	1    1650 5600
@@
 F 0 "J6" H 4720 4304 50  0000 R CNN
 F 1 "AVR-ISP-6" H 4720 4395 50  0000 R CNN
-F 2 "" V 4750 4350 50  0001 C CNN
+F 2 "Pin_Headers:Pin_Header_Straight_2x03_Pitch2.54mm" V 4750 4350 50  0001 C CNN
 F 3 " ~" H 3725 3750 50  0001 C CNN
 	1    5000 4300
@@
 F 0 "R14" H 3870 3946 50  0000 L CNN
 F 1 "100" H 3870 3855 50  0000 L CNN
-F 2 "" V 3730 3900 50  0001 C CNN
+F 2 "Resistors_SMD:R_0805_HandSoldering" V 3730 3900 50  0001 C CNN
 F 3 "~" H 3800 3900 50  0001 C CNN
 	1    3800 3900
@@
 F 0 "R16" H 4370 3946 50  0000 L CNN
 F 1 "100" H 4370 3855 50  0000 L CNN
-F 2 "" V 4230 3900 50  0001 C CNN
+F 2 "Resistors_SMD:R_0805_HandSoldering" V 4230 3900 50  0001 C CNN
 F 3 "~" H 4300 3900 50  0001 C CNN
 	1    4300 3900
@@
 F 0 "R15" H 4120 3946 50  0000 L CNN
 F 1 "100" H 4120 3855 50  0000 L CNN
-F 2 "" V 3980 3900 50  0001 C CNN
+F 2 "Resistors_SMD:R_0805_HandSoldering" V 3980 3900 50  0001 C CNN
 F 3 "~" H 4050 3900 50  0001 C CNN
 	1    4050 3900
@@
 F 0 "U8" H 9225 5287 60  0000 C CNN
 F 1 "HCPL2601SD" H 9225 5181 60  0000 C CNN
-F 2 "" H 9250 4800 60  0001 C CNN
+F 2 "lab_power_supply:HCPL2631SD" H 9250 4800 60  0001 C CNN
 F 3 "" H 9250 4800 60  0001 C CNN
 	1    9250 4850
@@
 F 0 "U6" H 7275 1313 60  0000 C CNN
 F 1 "HCPL2631SD" H 7275 1419 60  0000 C CNN
-F 2 "" H 7300 1700 60  0001 C CNN
+F 2 "lab_power_supply:HCPL2631SD" H 7300 1700 60  0001 C CNN
 F 3 "" H 7300 1700 60  0001 C CNN
 	1    7300 1750
@@
 F 0 "Q2" H 9155 1296 50  0000 L CNN
 F 1 "Q_NMOS_DGS" H 9155 1205 50  0000 L CNN
-F 2 "" H 9150 1350 50  0001 C CNN
+F 2 "TO_SOT_Packages_SMD:SuperSOT-3" H 9150 1350 50  0001 C CNN
 F 3 "~" H 8950 1250 50  0001 C CNN
 	1    8950 1250
@@
 F 0 "R10" V 8950 1050 50  0000 C CNN
 F 1 "330" V 9050 1100 50  0000 C CNN
-F 2 "" V 8930 900 50  0001 C CNN
+F 2 "Resistors_SMD:R_0805_HandSoldering" V 8930 900 50  0001 C CNN
 F 3 "~" H 9000 900 50  0001 C CNN
 	1    9000 900
@@
 F 0 "Q3" H 9155 2046 50  0000 L CNN
 F 1 "Q_NMOS_DGS" H 9155 1955 50  0000 L CNN
-F 2 "" H 9150 2100 50  0001 C CNN
+F 2 "TO_SOT_Packages_SMD:SuperSOT-3" H 9150 2100 50  0001 C CNN
 F 3 "~" H 8950 2000 50  0001 C CNN
 	1    8950 2000
@@
 F 0 "R11" V 8950 1800 50  0000 C CNN
 F 1 "330" V 9050 1850 50  0000 C CNN
-F 2 "" V 8930 1650 50  0001 C CNN
+F 2 "Resistors_SMD:R_0805_HandSoldering" V 8930 1650 50  0001 C CNN
 F 3 "~" H 9000 1650 50  0001 C CNN
 	1    9000 1650
@@
 F 0 "Q6" H 8155 5096 50  0000 L CNN
 F 1 "Q_NMOS_DGS" H 8155 5005 50  0000 L CNN
-F 2 "" H 8150 5150 50  0001 C CNN
+F 2 "TO_SOT_Packages_SMD:SuperSOT-3" H 8150 5150 50  0001 C CNN
 F 3 "~" H 7950 5050 50  0001 C CNN
 	1    7950 5050
@@
 F 0 "C17" H 9785 4804 50  0000 R CNN
 F 1 "0.1u" H 9785 4895 50  0000 R CNN
-F 2 "" H 9938 4700 50  0001 C CNN
+F 2 "Capacitors_SMD:C_0805_HandSoldering" H 9938 4700 50  0001 C CNN
 F 3 "~" H 9900 4850 50  0001 C CNN
 	1    9900 4850
@@
 F 0 "R18" H 8120 4696 50  0000 L CNN
 F 1 "500" H 8120 4605 50  0000 L CNN
-F 2 "" V 7980 4650 50  0001 C CNN
+F 2 "Resistors_SMD:R_0805_HandSoldering" V 7980 4650 50  0001 C CNN
 F 3 "~" H 8050 4650 50  0001 C CNN
 	1    8050 4650
@@
 F 0 "C12" H 6000 1700 50  0000 R CNN
 F 1 "0.1u" H 6050 1800 50  0000 R CNN
-F 2 "" H 5838 1600 50  0001 C CNN
+F 2 "Capacitors_SMD:C_0805_HandSoldering" H 5838 1600 50  0001 C CNN
 F 3 "~" H 5800 1750 50  0001 C CNN
 	1    5800 1750
@@
 F 0 "C15" V 2598 3700 50  0000 C CNN
 F 1 "C" V 2689 3700 50  0000 C CNN
-F 2 "" H 2888 3550 50  0001 C CNN
+F 2 "Capacitors_SMD:C_0805_HandSoldering" H 2888 3550 50  0001 C CNN
 F 3 "~" H 2850 3700 50  0001 C CNN
 	1    2850 3700
@@
 F 0 "U7" H 7275 2813 60  0000 C CNN
 F 1 "HCPL2631SD" H 7275 2919 60  0000 C CNN
-F 2 "" H 7300 3200 60  0001 C CNN
+F 2 "lab_power_supply:HCPL2631SD" H 7300 3200 60  0001 C CNN
 F 3 "" H 7300 3200 60  0001 C CNN
 	1    7300 3250
@@
 F 0 "Q4" H 9155 2796 50  0000 L CNN
 F 1 "Q_NMOS_DGS" H 9155 2705 50  0000 L CNN
-F 2 "" H 9150 2850 50  0001 C CNN
+F 2 "TO_SOT_Packages_SMD:SuperSOT-3" H 9150 2850 50  0001 C CNN
 F 3 "~" H 8950 2750 50  0001 C CNN
 	1    8950 2750
@@
 F 0 "R12" V 8950 2550 50  0000 C CNN
 F 1 "330" V 9050 2600 50  0000 C CNN
-F 2 "" V 8930 2400 50  0001 C CNN
+F 2 "Resistors_SMD:R_0805_HandSoldering" V 8930 2400 50  0001 C CNN
 F 3 "~" H 9000 2400 50  0001 C CNN
 	1    9000 2400
@@
 F 0 "Q5" H 9155 3546 50  0000 L CNN
 F 1 "Q_NMOS_DGS" H 9155 3455 50  0000 L CNN
-F 2 "" H 9150 3600 50  0001 C CNN
+F 2 "TO_SOT_Packages_SMD:SuperSOT-3" H 9150 3600 50  0001 C CNN
 F 3 "~" H 8950 3500 50  0001 C CNN
 	1    8950 3500
@@
 F 0 "R13" V 8950 3300 50  0000 C CNN
 F 1 "330" V 9050 3350 50  0000 C CNN
-F 2 "" V 8930 3150 50  0001 C CNN
+F 2 "Resistors_SMD:R_0805_HandSoldering" V 8930 3150 50  0001 C CNN
 F 3 "~" H 9000 3150 50  0001 C CNN
 	1    9000 3150
@@
 F 0 "C13" H 6000 3200 50  0000 R CNN
 F 1 "0.1u" H 6050 3300 50  0000 R CNN
-F 2 "" H 5838 3100 50  0001 C CNN
+F 2 "Capacitors_SMD:C_0805_HandSoldering" H 5838 3100 50  0001 C CNN
 F 3 "~" H 5800 3250 50  0001 C CNN
 	1    5800 3250
@@
 F 0 "J5" H 10300 1917 50  0000 C CNN
 F 1 "Isolated_ISP" H 10300 1826 50  0000 C CNN
-F 2 "" H 10250 1600 50  0001 C CNN
+F 2 "Pin_Headers:Pin_Header_Straight_1x08_Pitch2.54mm" H 10250 1600 50  0001 C CNN
 F 3 "~" H 10250 1600 50  0001 C CNN
 	1    10250 1600
@@
 F 0 "R23" H 3330 5704 50  0000 R CNN
 F 1 "10k" H 3330 5795 50  0000 R CNN
-F 2 "" V 3330 5750 50  0001 C CNN
+F 2 "Resistors_SMD:R_0805_HandSoldering" V 3330 5750 50  0001 C CNN
 F 3 "~" H 3400 5750 50  0001 C CNN
 	1    3400 5750
@@
 F 0 "R19" H 4270 5246 50  0000 L CNN
 F 1 "R" H 4270 5155 50  0000 L CNN
-F 2 "" V 4130 5200 50  0001 C CNN
+F 2 "Resistors_SMD:R_0805_HandSoldering" V 4130 5200 50  0001 C CNN
 F 3 "~" H 4200 5200 50  0001 C CNN
 	1    4200 5200
@@
 F 0 "R20" H 4520 5246 50  0000 L CNN
 F 1 "R" H 4520 5155 50  0000 L CNN
-F 2 "" V 4380 5200 50  0001 C CNN
+F 2 "Resistors_SMD:R_0805_HandSoldering" V 4380 5200 50  0001 C CNN
 F 3 "~" H 4450 5200 50  0001 C CNN
 	1    4450 5200
@@
 F 0 "R17" H 4620 3946 50  0000 L CNN
 F 1 "100" H 4620 3855 50  0000 L CNN
-F 2 "" V 4480 3900 50  0001 C CNN
+F 2 "Resistors_SMD:R_0805_HandSoldering" V 4480 3900 50  0001 C CNN
 F 3 "~" H 4550 3900 50  0001 C CNN
 	1    4550 3900
@@
 F 0 "J7" V 4200 5600 50  0000 L CNN
 F 1 "THERM0" V 4300 5400 50  0000 L CNN
-F 2 "" H 4200 5750 50  0001 C CNN
+F 2 "Pin_Headers:Pin_Header_Straight_1x02_Pitch2.54mm" H 4200 5750 50  0001 C CNN
 F 3 "~" H 4200 5750 50  0001 C CNN
 	1    4200 5750
@@
 F 0 "J8" V 4454 5830 50  0000 L CNN
 F 1 "THERM1" V 4550 5850 50  0000 L CNN
-F 2 "" H 4450 5750 50  0001 C CNN
+F 2 "Pin_Headers:Pin_Header_Straight_1x02_Pitch2.54mm" H 4450 5750 50  0001 C CNN
 F 3 "~" H 4450 5750 50  0001 C CNN
 	1    4450 5750
@@
 F 0 "C16" H 1700 4350 50  0000 L CNN
 F 1 "0.1u" H 1600 4250 50  0000 L CNN
-F 2 "" H 1938 4150 50  0001 C CNN
+F 2 "Capacitors_SMD:C_0805_HandSoldering" H 1938 4150 50  0001 C CNN
 F 3 "~" H 1900 4300 50  0001 C CNN
 	1    1900 4300
@@
 F 0 "U9" H 2000 3700 50  0000 C CNN
 F 1 "ATmega328PB-AU" H 2000 3800 50  0000 C CNN
-F 2 "Package_QFP:TQFP-32_7x7mm_P0.8mm" H 2600 5300 50  0001 C CIN
+F 2 "Housings_QFP:TQFP-32_7x7mm_Pitch0.8mm" H 2600 5300 50  0001 C CIN
 F 3 "http://ww1.microchip.com/downloads/en/DeviceDoc/40001906C.pdf" H 2600 5300 50  0001 C CNN
 	1    2600 5300

Commit message: pcb: Kaikki vedot tehty
Parts:
- C15: value C -> 0.1u
Connections:
- net labels added: GNDA
- wire segments 134 -> 133
Other:
- moved on the sheet: R19, R20

Commit message: Toinen konkka lisätty
Parts:
- J5: symbol lab_power_supply:Isolated_ISP -> pcb_1-rescue:Isolated_ISP-lab_power_supply
Changed lines of the file:
@@
 Connection ~ 7850 1800
 $Comp
-L lab_power_supply:Isolated_ISP J5
+L pcb_1-rescue:Isolated_ISP-lab_power_supply J5
 U 1 1 5DDDD6E5
 P 10250 1600
+AR Path="/5DDDD6E5" Ref="J5"  Part="1"
+AR Path="/5DD5EF4E/5DDDD6E5" Ref="J5"  Part="1"
 F 0 "J5" H 10300 1917 50  0000 C CNN
 F 1 "Isolated_ISP" H 10300 1826 50  0000 C CNN
@@
 	5800 3100 6900 3100
 $Comp
-L power:+5V #PWR?
+L power:+5V #PWR0103
 U 1 1 5E2C952E
 P 6900 2000
-F 0 "#PWR?" H 6900 1850 50  0001 C CNN
+F 0 "#PWR0103" H 6900 1850 50  0001 C CNN
 F 1 "+5V" H 6915 2173 50  0000 C CNN
 F 2 "" H 6900 2000 50  0001 C CNN
@@
 $EndComp
 $Comp
-L power:+5V #PWR?
+L power:+5V #PWR0104
 U 1 1 5E2CA1EB
 P 6900 3500
-F 0 "#PWR?" H 6900 3350 50  0001 C CNN
+F 0 "#PWR0104" H 6900 3350 50  0001 C CNN
 F 1 "+5V" H 6915 3673 50  0000 C CNN
 F 2 "" H 6900 3500 50  0001 C CNN
@@
 Connection ~ 6900 1900
 $Comp
-L power:GNDD #PWR?
+L power:GNDD #PWR0105
 U 1 1 5E2D403D
 P 6900 3000
-F 0 "#PWR?" H 6900 2750 50  0001 C CNN
+F 0 "#PWR0105" H 6900 2750 50  0001 C CNN
 F 1 "GNDD" H 6904 2845 50  0000 C CNN
 F 2 "" H 6900 3000 50  0001 C CNN
@@
 Connection ~ 6900 3100
 $Comp
-L power:GNDD #PWR?
+L power:GNDD #PWR0106
 U 1 1 5E2DDE26
 P 6900 1500
-F 0 "#PWR?" H 6900 1250 50  0001 C CNN
+F 0 "#PWR0106" H 6900 1250 50  0001 C CNN
 F 1 "GNDD" H 6904 1345 50  0000 C CNN
 F 2 "" H 6900 1500 50  0001 C CNN

Commit message: pcb: Rescue kirjasto poistettu
Parts:
- J5: symbol pcb_1-rescue:Isolated_ISP-lab_power_supply -> lab_power_supply:Isolated_ISP
Changed lines of the file:
@@
 Connection ~ 7850 1800
 $Comp
-L pcb_1-rescue:Isolated_ISP-lab_power_supply J5
+L lab_power_supply:Isolated_ISP J5
 U 1 1 5DDDD6E5
 P 10250 1600
