File: pcb_1/Micrcontroller.sch (KiCad schematic (older format))
At the start: 33 parts, among them J5 Isolated_ISP, J6 AVR-ISP-6, J7 THERM0, J8 THERM1, Q2 Q_NMOS_DGS, Q3 Q_NMOS_DGS, Q4 Q_NMOS_DGS, Q5 Q_NMOS_DGS, Q6 Q_NMOS_DGS, U6 HCPL2631SD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

Commit message: NMOS-symbolit muutettu
Parts:
- removed Q2, Q3, Q4, Q5, Q6: Q_NMOS_DGS, TO_SOT_Packages_SMD:SuperSOT-3, symbol Device:Q_NMOS_DGS
- added Q2, Q3, Q4, Q5, Q6: Q_NMOS_GSD, TO_SOT_Packages_SMD:SuperSOT-3, symbol Device:Q_NMOS_GSD
Changed lines of the file:
@@
 	6900 1800 6650 1800
-$Comp
-L Device:Q_NMOS_DGS Q2
-U 1 1 5DDEB268
-P 8950 1250
-F 0 "Q2" H 9155 1296 50  0000 L CNN
-F 1 "Q_NMOS_DGS" H 9155 1205 50  0000 L CNN
-F 2 "TO_SOT_Packages_SMD:SuperSOT-3" H 9150 1350 50  0001 C CNN
-F 3 "~" H 8950 1250 50  0001 C CNN
-	1    8950 1250
-	-1   0    0    -1
-$EndComp
 $Comp
 L Device:R R10
@@
 	8850 900  8850 1050
 $Comp
-L Device:Q_NMOS_DGS Q3
-U 1 1 5DDF29F3
-P 8950 2000
-F 0 "Q3" H 9155 2046 50  0000 L CNN
-F 1 "Q_NMOS_DGS" H 9155 1955 50  0000 L CNN
-F 2 "TO_SOT_Packages_SMD:SuperSOT-3" H 9150 2100 50  0001 C CNN
-F 3 "~" H 8950 2000 50  0001 C CNN
-	1    8950 2000
-	-1   0    0    -1
-$EndComp
-$Comp
 L Device:R R11
 U 1 1 5DDF29FD
@@
 Connection ~ 8850 900
 $Comp
-L Device:Q_NMOS_DGS Q6
-U 1 1 5DE3498E
-P 7950 5050
-F 0 "Q6" H 8155 5096 50  0000 L CNN
-F 1 "Q_NMOS_DGS" H 8155 5005 50  0000 L CNN
-F 2 "TO_SOT_Packages_SMD:SuperSOT-3" H 8150 5150 50  0001 C CNN
-F 3 "~" H 7950 5050 50  0001 C CNN
-	1    7950 5050
-	1    0    0    -1
-$EndComp
-$Comp
 L power:GNDD #PWR026
 U 1 1 5DE46C99
@@
 	6900 3300 6650 3300
 $Comp
-L Device:Q_NMOS_DGS Q4
-U 1 1 5DDA674F
-P 8950 2750
-F 0 "Q4" H 9155 2796 50  0000 L CNN
-F 1 "Q_NMOS_DGS" H 9155 2705 50  0000 L CNN
-F 2 "TO_SOT_Packages_SMD:SuperSOT-3" H 9150 2850 50  0001 C CNN
-F 3 "~" H 8950 2750 50  0001 C CNN
-	1    8950 2750
-	-1   0    0    -1
-$EndComp
-$Comp
 L Device:R R12
 U 1 1 5DDA6759
@@
 	8850 2400 8850 2550
 $Comp
-L Device:Q_NMOS_DGS Q5
-U 1 1 5DDA6764
-P 8950 3500
-F 0 "Q5" H 9155 3546 50  0000 L CNN
-F 1 "Q_NMOS_DGS" H 9155 3455 50  0000 L CNN
-F 2 "TO_SOT_Packages_SMD:SuperSOT-3" H 9150 3600 50  0001 C CNN
-F 3 "~" H 8950 3500 50  0001 C CNN
-	1    8950 3500
-	-1   0    0    -1
-$EndComp
-$Comp
 L Device:R R13
 U 1 1 5DDA676E
@@
 Wire Wire Line
 	9400 3150 9150 3150
-Wire Wire Line
-	8850 2950 9300 2950
 Wire Wire Line
 	7750 3300 7850 3300
@@
 Connection ~ 9900 5000
 Connection ~ 11050 3900
+Wire Wire Line
+	8850 2950 9300 2950
+$Comp
+L Device:Q_NMOS_GSD Q6
+U 1 1 5DD7D321
+P 8950 3500
+F 0 "Q6" H 9156 3546 50  0000 L CNN
+F 1 "Q_NMOS_GSD" H 9156 3455 50  0000 L CNN
+F 2 "TO_SOT_Packages_SMD:SuperSOT-3" H 9150 3600 50  0001 C CNN
+F 3 "~" H 8950 3500 50  0001 C CNN
+	1    8950 3500
+	-1   0    0    -1
+$EndComp
+$Comp
+L Device:Q_NMOS_GSD Q5
+U 1 1 5DD80C3B
+P 8950 2750
+F 0 "Q5" H 9156 2796 50  0000 L CNN
+F 1 "Q_NMOS_GSD" H 9156 2705 50  0000 L CNN
+F 2 "TO_SOT_Packages_SMD:SuperSOT-3" H 9150 2850 50  0001 C CNN
+F 3 "~" H 8950 2750 50  0001 C CNN
+	1    8950 2750
+	-1   0    0    -1
+$EndComp
+$Comp
+L Device:Q_NMOS_GSD Q3
+U 1 1 5DD817D8
+P 8950 1250
+F 0 "Q3" H 9156 1296 50  0000 L CNN
+F 1 "Q_NMOS_GSD" H 9156 1205 50  0000 L CNN
+F 2 "TO_SOT_Packages_SMD:SuperSOT-3" H 9150 1350 50  0001 C CNN
+F 3 "~" H 8950 1250 50  0001 C CNN
+	1    8950 1250
+	-1   0    0    -1
+$EndComp
+$Comp
+L Device:Q_NMOS_GSD Q4
+U 1 1 5DD82392
+P 8950 2000
+F 0 "Q4" H 9156 2046 50  0000 L CNN
+F 1 "Q_NMOS_GSD" H 9156 1955 50  0000 L CNN
+F 2 "TO_SOT_Packages_SMD:SuperSOT-3" H 9150 2100 50  0001 C CNN
+F 3 "~" H 8950 2000 50  0001 C CNN
+	1    8950 2000
+	-1   0    0    -1
+$EndComp
+$Comp
+L Device:Q_NMOS_GSD Q2
+U 1 1 5DD82DD0
+P 7950 5050
+F 0 "Q2" H 8156 5096 50  0000 L CNN
+F 1 "Q_NMOS_GSD" H 8156 5005 50  0000 L CNN
+F 2 "TO_SOT_Packages_SMD:SuperSOT-3" H 8150 5150 50  0001 C CNN
+F 3 "~" H 7950 5050 50  0001 C CNN
+	1    7950 5050
+	1    0    0    -1
+$EndComp
 $EndSCHEMATC

Commit message: pcb: Silkscreeniä päivitetty
Connections:
- wire segments 133 -> 134
Changed lines of the file:
@@
 	1    0    0    -1
 $EndComp
-Wire Wire Line
-	4200 5300 4200 5450
 Connection ~ 4200 5300
 Wire Wire Line
@@
 	4450 5400 4450 5450
 Connection ~ 4450 5400
-Wire Wire Line
-	4450 5250 4450 5400
 Wire Wire Line
 	4200 5250 4200 5300
@@
 	4550 3750 4550 3650
 NoConn ~ 3200 5800
-$Comp
-L Connector_Generic:Conn_02x01 J7
-U 1 1 5DE6EFB6
-P 4450 5650
-F 0 "J7" V 4450 5750 50  0000 L CNN
-F 1 "THERM0" V 4550 5750 50  0000 L CNN
-F 2 "Pin_Headers:Pin_Header_Straight_1x02_Pitch2.54mm" H 4450 5650 50  0001 C CNN
-F 3 "~" H 4450 5650 50  0001 C CNN
-	1    4450 5650
-	0    1    1    0
-$EndComp
-$Comp
-L Connector_Generic:Conn_02x01 J8
-U 1 1 5DE6FB9D
-P 4200 5650
-F 0 "J8" V 4200 5500 50  0000 L CNN
-F 1 "THERM1" V 4300 5300 50  0000 L CNN
-F 2 "Pin_Headers:Pin_Header_Straight_1x02_Pitch2.54mm" H 4200 5650 50  0001 C CNN
-F 3 "~" H 4200 5650 50  0001 C CNN
-	1    4200 5650
-	0    1    1    0
-$EndComp
 Connection ~ 9900 4700
 $Comp
@@
 	1    0    0    -1
 $EndComp
+Wire Wire Line
+	4450 5250 4450 5350
+$Comp
+L Connector_Generic:Conn_02x01 J7
+U 1 1 5DE6EFB6
+P 4450 5750
+F 0 "J7" V 4450 5600 50  0000 L CNN
+F 1 "THERM0" V 4550 5400 50  0000 L CNN
+F 2 "Pin_Headers:Pin_Header_Straight_1x02_Pitch2.54mm" H 4450 5750 50  0001 C CNN
+F 3 "~" H 4450 5750 50  0001 C CNN
+	1    4450 5750
+	0    -1   -1   0
+$EndComp
+$Comp
+L Connector_Generic:Conn_02x01 J8
+U 1 1 5DE6FB9D
+P 4200 5750
+F 0 "J8" V 4200 5850 50  0000 L CNN
+F 1 "THERM1" V 4300 5850 50  0000 L CNN
+F 2 "Pin_Headers:Pin_Header_Straight_1x02_Pitch2.54mm" H 4200 5750 50  0001 C CNN
+F 3 "~" H 4200 5750 50  0001 C CNN
+	1    4200 5750
+	0    -1   -1   0
+$EndComp
+Wire Wire Line
+	4200 5300 4200 5450
+Connection ~ 4450 5350
+Wire Wire Line
+	4450 5350 4450 5400
 $EndSCHEMATC

Commit message: pcb: Gerber tiedostot lisätty
Parts:
- added J9: CS, Connector_PinHeader_2.54mm:PinHeader_1x01_P2.54mm_Vertical, symbol Connector_Generic:Conn_01x01
- added R25: 100, Resistor_SMD:R_0805_2012Metric_Pad1.15x1.40mm_HandSolder, symbol Device:R
Connections:
- wire segments 134 -> 135
Changed lines of the file:
@@
 SLAVE_CS
 Wire Wire Line
-	3300 3650 3300 4300
+	3300 3650 3300 3850
 Wire Wire Line
 	6650 1700 6900 1700
@@
 Wire Wire Line
 	4450 5400 4450 5450
-Connection ~ 4450 5400
 Wire Wire Line
 	4200 5250 4200 5300
@@
 	1    0    0    -1
 $EndComp
-Wire Wire Line
-	4450 5250 4450 5350
 $Comp
 L Connector_Generic:Conn_02x01 J7
@@
 Wire Wire Line
 	4200 5300 4200 5450
+$Comp
+L Device:R R25
+U 1 1 5DDD49CA
+P 3450 3850
+F 0 "R25" H 3520 3896 50  0000 L CNN
+F 1 "100" H 3520 3805 50  0000 L CNN
+F 2 "Resistor_SMD:R_0805_2012Metric_Pad1.15x1.40mm_HandSolder" V 3380 3850 50  0001 C CNN
+F 3 "~" H 3450 3850 50  0001 C CNN
+	1    3450 3850
+	0    1    1    0
+$EndComp
+Connection ~ 3300 3850
+Wire Wire Line
+	3300 3850 3300 4300
+$Comp
+L Connector_Generic:Conn_01x01 J9
+U 1 1 5DDD56A7
+P 3600 3650
+F 0 "J9" V 3700 3700 50  0000 R CNN
+F 1 "CS" V 3600 3850 50  0000 R CNN
+F 2 "Connector_PinHeader_2.54mm:PinHeader_1x01_P2.54mm_Vertical" H 3600 3650 50  0001 C CNN
+F 3 "~" H 3600 3650 50  0001 C CNN
+	1    3600 3650
+	0    -1   -1   0
+$EndComp
+Connection ~ 4450 5400
+Wire Wire Line
+	4450 5350 4450 5400
 Connection ~ 4450 5350
 Wire Wire Line
-	4450 5350 4450 5400
+	4450 5250 4450 5350
 $EndSCHEMATC

Commit message: pcb: Kondensaattoreiden footprintit muuttettu
Parts:
- C12, C13, C14, C15, C16, C17: footprint Capacitors_SMD:C_0805_HandSoldering -> Capacitor_SMD:C_0805_2012Metric_Pad1.15x1.40mm_HandSolder
Connections:
- wire segments 135 -> 134
Changed lines of the file:
@@
 F 0 "C14" V 2148 3700 50  0000 C CNN
 F 1 "0.1u" V 2239 3700 50  0000 C CNN
-F 2 "Capacitors_SMD:C_0805_HandSoldering" H 2438 3550 50  0001 C CNN
+F 2 "Capacitor_SMD:C_0805_2012Metric_Pad1.15x1.40mm_HandSolder" H 2438 3550 50  0001 C CNN
 F 3 "~" H 2400 3700 50  0001 C CNN
 	1    2400 3700
@@
 F 0 "C17" H 9785 4804 50  0000 R CNN
 F 1 "0.1u" H 9785 4895 50  0000 R CNN
-F 2 "Capacitors_SMD:C_0805_HandSoldering" H 9938 4700 50  0001 C CNN
+F 2 "Capacitor_SMD:C_0805_2012Metric_Pad1.15x1.40mm_HandSolder" H 9938 4700 50  0001 C CNN
 F 3 "~" H 9900 4850 50  0001 C CNN
 	1    9900 4850
@@
 F 0 "C12" H 6000 1700 50  0000 R CNN
 F 1 "0.1u" H 6050 1800 50  0000 R CNN
-F 2 "Capacitors_SMD:C_0805_HandSoldering" H 5838 1600 50  0001 C CNN
+F 2 "Capacitor_SMD:C_0805_2012Metric_Pad1.15x1.40mm_HandSolder" H 5838 1600 50  0001 C CNN
 F 3 "~" H 5800 1750 50  0001 C CNN
 	1    5800 1750
@@
 F 0 "C15" V 2598 3700 50  0000 C CNN
 F 1 "0.1u" V 2689 3700 50  0000 C CNN
-F 2 "Capacitors_SMD:C_0805_HandSoldering" H 2888 3550 50  0001 C CNN
+F 2 "Capacitor_SMD:C_0805_2012Metric_Pad1.15x1.40mm_HandSolder" H 2888 3550 50  0001 C CNN
 F 3 "~" H 2850 3700 50  0001 C CNN
 	1    2850 3700
@@
 F 0 "C13" H 6000 3200 50  0000 R CNN
 F 1 "0.1u" H 6050 3300 50  0000 R CNN
-F 2 "Capacitors_SMD:C_0805_HandSoldering" H 5838 3100 50  0001 C CNN
+F 2 "Capacitor_SMD:C_0805_2012Metric_Pad1.15x1.40mm_HandSolder" H 5838 3100 50  0001 C CNN
 F 3 "~" H 5800 3250 50  0001 C CNN
 	1    5800 3250
@@
 F 0 "C16" H 1700 4350 50  0000 L CNN
 F 1 "0.1u" H 1600 4250 50  0000 L CNN
-F 2 "Capacitors_SMD:C_0805_HandSoldering" H 1938 4150 50  0001 C CNN
+F 2 "Capacitor_SMD:C_0805_2012Metric_Pad1.15x1.40mm_HandSolder" H 1938 4150 50  0001 C CNN
 F 3 "~" H 1900 4300 50  0001 C CNN
 	1    1900 4300
@@
 Connection ~ 4450 5400
 Wire Wire Line
-	4450 5350 4450 5400
-Connection ~ 4450 5350
-Wire Wire Line
-	4450 5250 4450 5350
+	4450 5250 4450 5400
 $EndSCHEMATC

Commit message: pcb: Optcouplereitten virranrajotinvastkset muutettu
Parts:
- R10, R11, R12, R13: value 330 -> 360
- R18: value 500 -> 360
Changed lines of the file:
@@
 P 9000 900
 F 0 "R10" V 8950 1050 50  0000 C CNN
-F 1 "330" V 9050 1100 50  0000 C CNN
+F 1 "360" V 9050 1100 50  0000 C CNN
 F 2 "Resistors_SMD:R_0805_HandSoldering" V 8930 900 50  0001 C CNN
 F 3 "~" H 9000 900 50  0001 C CNN
@@
 P 9000 1650
 F 0 "R11" V 8950 1800 50  0000 C CNN
-F 1 "330" V 9050 1850 50  0000 C CNN
+F 1 "360" V 9050 1850 50  0000 C CNN
 F 2 "Resistors_SMD:R_0805_HandSoldering" V 8930 1650 50  0001 C CNN
 F 3 "~" H 9000 1650 50  0001 C CNN
@@
 P 8050 4650
 F 0 "R18" H 8120 4696 50  0000 L CNN
-F 1 "500" H 8120 4605 50  0000 L CNN
+F 1 "360" H 8120 4605 50  0000 L CNN
 F 2 "Resistors_SMD:R_0805_HandSoldering" V 7980 4650 50  0001 C CNN
 F 3 "~" H 8050 4650 50  0001 C CNN
@@
 P 9000 2400
 F 0 "R12" V 8950 2550 50  0000 C CNN
-F 1 "330" V 9050 2600 50  0000 C CNN
+F 1 "360" V 9050 2600 50  0000 C CNN
 F 2 "Resistors_SMD:R_0805_HandSoldering" V 8930 2400 50  0001 C CNN
 F 3 "~" H 9000 2400 50  0001 C CNN
@@
 P 9000 3150
 F 0 "R13" V 8950 3300 50  0000 C CNN
-F 1 "330" V 9050 3350 50  0000 C CNN
+F 1 "360" V 9050 3350 50  0000 C CNN
 F 2 "Resistors_SMD:R_0805_HandSoldering" V 8930 3150 50  0001 C CNN
 F 3 "~" H 9000 3150 50  0001 C CNN
